File: CAN-Acquisition-Module_MCU.sch (KiCad schematic (older format))
At the start: 11 parts

Commit message: Schematic started
MCU section well advanced, power section started as well
Parts:
- added C? (x2): 20 pF, Capacitor_SMD:C_0603_1608Metric, symbol Device:C_Small
- added C?: 100 nF, Capacitor_SMD:C_0402_1005Metric, symbol Device:C_Small
- added C?: 1 uF, Capacitor_SMD:C_0603_1608Metric, symbol Device:C_Small
- added H? (x4): MountingHole, symbol Mechanical:MountingHole
- added J?: Conn_02x05_Odd_Even, symbol Connector_Generic:Conn_02x05_Odd_Even
- added L? (x2): Ferrite, Inductor_SMD:L_0603_1608Metric, symbol Device:L_Small
- added Y?: Crystal_GND24_Small, Crystal:Crystal_SMD_3225-4Pin_3.2x2.5mm, symbol Device:Crystal_GND24_Small
Connections:
- net GND: now also C?.1, C?.2, J?.10 (Pin_10), L?.1, Y?.2, Y?.4
- net at U?.16 (PF.3): now also C?.2, Y?.3
- net at U?.17 (PF.2): now also C?.1, Y?.1
- net nRESET: now reaches C?.1, R?.2, U?.32 (nRESET)
- net nRESET: now also J?.8 (Pin_8)
- net ICE_DAT: now reaches U?.33 (PF.0)
- net ICE_DAT: now also J?.4 (Pin_4)
- net ICE_CLK: now reaches U?.34 (PF.1)
- net ICE_CLK: now also J?.6 (Pin_6)
- net UART0_TX: now reaches U?.55 (PB.13)
- net UART0_TX: now also J?.7 (Pin_7)
- net UART0_RX: now reaches U?.56 (PB.12)
- net UART0_RX: now also J?.9 (Pin_9)
- net +3.3VA: now reaches U?.57 (AVDD)
- net +3.3VA: now also C?.1, C?.1, L?.2
- net +1V8: now reaches U?.58 (VREF)
- net GNDA: now reaches U?.59 (AVSS)
- net GNDA: now also C?.2, C?.2, L?.2
- net VDD renamed +3V3
- net +3V3: now also J?.2 (Pin_2), L?.1
Other:
- note added: "Place next to pin 57"
- note added: "Programming connector"
- note removed: "Programming connector!"
- moved on the sheet: C?, R?
