File: CAN-Acquisition-Module_Screen.kicad_sch (KiCad schematic)
At the start: 0 parts

Commit message: Added analog and sensors sections
Other:
- company: (none) -> École de Technologie Supérieure - Laboratoire thermique et science du bâtiment (LTSB)
- title: (none) -> CANbus Acquisition Module
Changed lines of the file:
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@@
 (kicad_sch (version 20211123) (generator eeschema)
   (paper "A4")
+  (title_block
+    (title "CANbus Acquisition Module")
+    (date "2022-06-01")
+    (rev "A1")
+    (company "École de Technologie Supérieure - Laboratoire thermique et science du bâtiment (LTSB)")
+    (comment 1 "Designer: Hugo Boyce")
+  )
 )
