File: CAN-Acquisition-Module_LED.kicad_sch (KiCad schematic)
At the start: 4 parts

Commit message: Added analog and sensors sections
Other:
- company: (none) -> École de Technologie Supérieure - Laboratoire thermique et science du bâtiment (LTSB)
- title: (none) -> CANbus Acquisition Module
Changed lines of the file:
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@@
 (kicad_sch (version 20211123) (generator eeschema)
   (paper "A4")
+  (title_block
+    (title "CANbus Acquisition Module")
+    (date "2022-06-01")
+    (rev "A1")
+    (company "École de Technologie Supérieure - Laboratoire thermique et science du bâtiment (LTSB)")
+    (comment 1 "Designer: Hugo Boyce")
+  )
   (wire (pts (xy 88.9 58.42) (xy 88.9 63.5))
     (stroke (width 0) (type default) (color 0 0 0 0))

Commit message: Added screen sections and annotations
Parts:
- removed D?: LED_RGBA, symbol Device:LED_RGBA
- removed R? (x2): 120 Ω, Resistor_SMD:R_0603_1608Metric, symbol Device:R_Small_US
- removed R?: 300 Ω, Resistor_SMD:R_0603_1608Metric, symbol Device:R_Small_US
Changed lines of the file:
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@@
     (comment 1 "Designer: Hugo Boyce")
   )
-  (wire (pts (xy 88.9 58.42) (xy 88.9 63.5))
-    (stroke (width 0) (type default) (color 0 0 0 0))
-  )
-  (wire (pts (xy 93.98 58.42) (xy 93.98 63.5))
-    (stroke (width 0) (type default) (color 0 0 0 0))
-  )
-  (wire (pts (xy 88.9 68.58) (xy 88.9 74.93))
-    (stroke (width 0) (type default) (color 0 0 0 0))
-  )
-  (wire (pts (xy 99.06 68.58) (xy 99.06 74.93))
-    (stroke (width 0) (type default) (color 0 0 0 0))
-  )
-  (wire (pts (xy 93.98 68.58) (xy 93.98 74.93))
-    (stroke (width 0) (type default) (color 0 0 0 0))
-  )
-  (wire (pts (xy 99.06 58.42) (xy 99.06 63.5))
-    (stroke (width 0) (type default) (color 0 0 0 0))
-  )
-  (hierarchical_label "LED_B" (shape input) (at 99.06 74.93 270)
-    (effects (font (size 1.27 1.27)) (justify right))
-  )
-  (hierarchical_label "LED_R" (shape input) (at 88.9 74.93 270)
-    (effects (font (size 1.27 1.27)) (justify right))
-  )
-  (hierarchical_label "LED_G" (shape input) (at 93.98 74.93 270)
-    (effects (font (size 1.27 1.27)) (justify right))
-  )
-  (symbol (lib_id "power:+3.3V") (at 93.98 48.26 0) (unit 1)
-    (in_bom yes) (on_board yes) (fields_autoplaced)
-    (property "Reference" "#PWR?" (id 0) (at 93.98 52.07 0)
-      (effects (font (size 1.27 1.27)) hide)
-    )
-    (property "Value" "+3.3V" (id 1) (at 93.98 44.6842 0))
-    (property "Footprint" "" (id 2) (at 93.98 48.26 0)
-      (effects (font (size 1.27 1.27)) hide)
-    )
-    (property "Datasheet" "" (id 3) (at 93.98 48.26 0)
-      (effects (font (size 1.27 1.27)) hide)
-    )
-    (pin "1")
-  )
-  (symbol (lib_id "Device:R_Small_US") (at 93.98 66.04 180) (unit 1)
-    (in_bom yes) (on_board yes)
-    (property "Reference" "R?" (id 0) (at 92.71 62.23 90)
-      (effects (font (size 1.27 1.27)) (justify left))
-    )
-    (property "Value" "120 Ω" (id 1) (at 95.25 67.31 90)
-      (effects (font (size 1.27 1.27)) (justify left))
-    )
-    (property "Footprint" "Resistor_SMD:R_0603_1608Metric" (id 2) (at 93.98 66.04 0)
-      (effects (font (size 1.27 1.27)) hide)
-    )
-    (property "Datasheet" "~" (id 3) (at 93.98 66.04 0)
-      (effects (font (size 1.27 1.27)) hide)
-    )
-    (pin "1")
-    (pin "2")
-  )
-  (symbol (lib_id "Device:R_Small_US") (at 88.9 66.04 180) (unit 1)
-    (in_bom yes) (on_board yes)
-    (property "Reference" "R?" (id 0) (at 87.63 62.23 90)
-      (effects (font (size 1.27 1.27)) (justify left))
-    )
-    (property "Value" "300 Ω" (id 1) (at 90.17 67.31 90)
-      (effects (font (size 1.27 1.27)) (justify left))
-    )
-    (property "Footprint" "Resistor_SMD:R_0603_1608Metric" (id 2) (at 88.9 66.04 0)
-      (effects (font (size 1.27 1.27)) hide)
-    )
-    (property "Datasheet" "~" (id 3) (at 88.9 66.04 0)
-      (effects (font (size 1.27 1.27)) hide)
-    )
-    (pin "1")
-    (pin "2")
-  )
-  (symbol (lib_id "Device:R_Small_US") (at 99.06 66.04 180) (unit 1)
-    (in_bom yes) (on_board yes)
-    (property "Reference" "R?" (id 0) (at 97.79 62.23 90)
-      (effects (font (size 1.27 1.27)) (justify left))
-    )
-    (property "Value" "120 Ω" (id 1) (at 100.33 67.31 90)
-      (effects (font (size 1.27 1.27)) (justify left))
-    )
-    (property "Footprint" "Resistor_SMD:R_0603_1608Metric" (id 2) (at 99.06 66.04 0)
-      (effects (font (size 1.27 1.27)) hide)
-    )
-    (property "Datasheet" "~" (id 3) (at 99.06 66.04 0)
-      (effects (font (size 1.27 1.27)) hide)
-    )
-    (pin "1")
-    (pin "2")
-  )
-  (symbol (lib_id "Device:LED_RGBA") (at 93.98 53.34 90) (unit 1)
-    (in_bom yes) (on_board yes) (fields_autoplaced)
-    (property "Reference" "D?" (id 0) (at 102.362 52.5053 90)
-      (effects (font (size 1.27 1.27)) (justify right))
-    )
-    (property "Value" "LED_RGBA" (id 1) (at 102.362 55.0422 90)
-      (effects (font (size 1.27 1.27)) (justify right))
-    )
-    (property "Footprint" "" (id 2) (at 95.25 53.34 0)
-      (effects (font (size 1.27 1.27)) hide)
-    )
-    (property "Datasheet" "~" (id 3) (at 95.25 53.34 0)
-      (effects (font (size 1.27 1.27)) hide)
-    )
-    (pin "1")
-    (pin "2")
-    (pin "3")
-    (pin "4")
-  )
 )
