File: CAN-Acquisition-Module.kicad_pcb (KiCad board)
At the start: 4 copper layers, 95 x 65 mm, 211 parts, among them J1 Conn_01x04, J10 OSTVN04A150, J11 OSTVN04A150, J12 OSTVN04A150, J13 OSTVN04A150, J2 Conn_01x02, J3 Conn_01x03, J4 Conn_02x05_Odd_Even, J5 OSTVN04A150, J6 OSTVN04A150, J7 USB_B_Micro, J8 OSTVN04A150, J9 OSTVN04A150, Q1 SI2318A, U1 AZ431LAN, U10 BD12734FVJ-E2, U2 S-8581AA, U3 M483SGCAE, U4 SN65HVD234, U5 BD12734FVJ-E2, U6 SCD30, U7 SHT35-DIS, U8 OPA4317IPWR, U9 ERC13232FN-1, Y1 12 MHz

Commit message: Rev. A1 release
Parts:
- added C32: 100 nF, Capacitor_SMD:C_0402_1005Metric, F.Cu at (94.4, 53.4)
- added G1: LOGO, LOGO, F.Cu at (101.5, 57.1)
- added G2: LOGO, LOGO, F.Cu at (45.0, 51.6)
- added G5: LOGO, LOGO, B.Cu at (53.4, 40.1)
- added G5: LOGO, LOGO, B.Cu at (82.1, 40.1)
- added R13: 10 kΩ, Resistor_SMD:R_0603_1608Metric, F.Cu at (90.9, 52.4)
- added R14: 10 kΩ, Resistor_SMD:R_0603_1608Metric, F.Cu at (105.4, 48.0)
- added U4: SST25VF080B-50-4x-S2Ax, CAN-Acquisition-Module:SOIC-8_P1.27mm_Multi, F.Cu at (98.2, 49.7)
- moved C36 24.3 mm to (83.6, 36.0), turned to 90 degrees
- moved C37 22.7 mm to (84.8, 36.0), turned to 90 degrees
- moved U5 16.9 mm to (89.0, 36.0), turned to 0 degrees
- moved R20 9.82 mm to (90.8, 40.9), turned to 90 degrees
- moved R18 9.47 mm to (95.5, 34.8), turned to 0 degrees
- moved C39 8.51 mm to (95.7, 41.4)
- moved R23 8.51 mm to (94.2, 44.4)
- moved R24 8.51 mm to (94.2, 41.4)
- moved R25 8.51 mm to (95.7, 44.4)
- moved C38 8.13 mm to (92.3, 40.9), turned to 90 degrees
- moved R17 7.73 mm to (95.5, 37.0), turned to 0 degrees
- moved NT1 7.61 mm to (67.0, 31.2), turned to 0 degrees
- moved R21 5.87 mm to (98.6, 38.1), turned to -90 degrees
- moved C33 5.10 mm to (99.3, 35.8), turned to 0 degrees
- moved R19 3.79 mm to (90.8, 43.9), turned to 90 degrees
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- renumbered C32 to C33, C33 to C34, C34 to C35, C35 to C36, C36 to C37, C37 to C38, C38 to C39, C39 to C40, C40 to C41, C41 to C42, C42 to C43, C43 to C44, C44 to C45, C45 to C46, C46 to C47, C47 to C48, C48 to C49, C49 to C50, C50 to C51, C51 to C52, C52 to C53, C53 to C54, C54 to C55, C55 to C56, C56 to C57, C57 to C58, C58 to C59, C59 to C60, C60 to C61, C61 to C62, C62 to C63, C63 to C64, C64 to C65, C65 to C66, C66 to C67, C67 to C68, R13 to R15, R14 to R16, R15 to R17, R16 to R18, R17 to R19, R18 to R20, R19 to R21, R20 to R22, R21 to R23, R22 to R24, R23 to R25, R24 to R26, R25 to R27, R26 to R28, R27 to R29, R28 to R30, R29 to R31, R30 to R32, R31 to R33, R32 to R34, R33 to R35, R34 to R36, R35 to R37, R36 to R38, R37 to R39, R38 to R40, R39 to R41, R40 to R42, R41 to R43, R42 to R44, R43 to R45, R44 to R46, R45 to R47, R46 to R48, R47 to R49, R48 to R50, R49 to R51, R50 to R52, R51 to R53, R52 to R54, R53 to R55, R54 to R56, R55 to R57, R56 to R58, R57 to R59, R58 to R60, R59 to R61, R60 to R62, R61 to R63, R62 to R64, R63 to R65, R64 to R66, R65 to R67, R66 to R68, R67 to R69, R68 to R70, R69 to R71, R70 to R72, R71 to R73, R72 to R74, R73 to R75, R74 to R76, R75 to R77, R76 to R78, R77 to R79, R78 to R80, R79 to R81, U9 to U10, U10 to U11, U4 to U5, U5 to U6, U6 to U7, U7 to U8, U8 to U9
Connections:
- C7 pad 1: Net-(C6-Pad1) -> Net-(C7-Pad1)
- C8 pad 1: Net-(C6-Pad1) -> Net-(C7-Pad1)
- NT1 pad 2: Net-(NT1-Pad2) -> Net-(C7-Pad1)
- R68 pad 2: /ADC9 -> /ADC8
- R69 pad 2: /ADC10 -> /ADC11
- R70 pad 2: /ADC11 -> /ADC10
- R71 pad 2: /ADC8 -> /ADC9
- U11 pad 1: /ADC4 -> /ADC5
- U11 pad 13: /ADC7 -> /ADC6
- U11 pad 14: /ADC7 -> /ADC6
- U11 pad 2: /ADC4 -> /ADC5
- U11 pad 6: /ADC5 -> /ADC4
- U11 pad 7: /ADC5 -> /ADC4
- U11 pad 8: /ADC6 -> /ADC7
- U11 pad 9: /ADC6 -> /ADC7
- U2 pad 1: Net-(NT1-Pad2) -> Net-(C7-Pad1)
- U2 pad 3: Net-(NT1-Pad2) -> Net-(C7-Pad1)
- U3 pad 18: unconnected-(U3-Pad18) -> /MCU/MEM_MISO
- U3 pad 19: unconnected-(U3-Pad19) -> /MCU/MEM_MOSI
- U3 pad 20: unconnected-(U3-Pad20) -> /MCU/MEM_CLK
- U3 pad 21: unconnected-(U3-Pad21) -> /MCU/MEM_nSS
- U6 pad 1: /ADC0 -> /ADC1
- U6 pad 13: /ADC3 -> /ADC2
- U6 pad 14: /ADC3 -> /ADC2
- U6 pad 2: /ADC0 -> /ADC1
- U6 pad 6: /ADC1 -> /ADC0
- U6 pad 7: /ADC1 -> /ADC0
- U6 pad 8: /ADC2 -> /ADC3
- U6 pad 9: /ADC2 -> /ADC3
- U9 pad 1: /ADC8 -> /ADC9
- U9 pad 14: /ADC11 -> /ADC10
- U9 pad 7: /ADC9 -> /ADC8
- U9 pad 8: /ADC10 -> /ADC11
Routing:
- net +3V3: track 326.4 -> 380.7 mm, vias 20 -> 22
- net /MCU/MEM_nSS: track 0.00 -> 30.3 mm, vias 0 -> 2
- net /MCU/MEM_MISO: track 0.00 -> 26.5 mm
- net /CANbus/CAN_TX: track 0.00 -> 25.3 mm
- net /CANbus/CAN_H/YEL: track 93.3 -> 117.7 mm
- net /CANbus/CAN_PIN5: track 0.00 -> 23.8 mm, vias 0 -> 2
- net /CANbus/CAN_L/GRN: track 93.8 -> 116.5 mm
- net /CANbus/CAN_RX: track 0.00 -> 19.7 mm
- net /CANbus/CAN_PIN8: track 0.00 -> 18.5 mm, vias 0 -> 2
- net Net-(C39-Pad1): track 0.00 -> 17.4 mm, vias 0 -> 2
- net /MCU/MEM_CLK: track 0.00 -> 16.1 mm, vias 0 -> 2
- net /MCU/MEM_MOSI: track 0.00 -> 14.4 mm
- net Net-(C38-Pad1): track 0.00 -> 14.2 mm
- net /ADC1: track 12.4 -> 19.3 mm, vias 0 -> 2
- net /ADC11: track 48.5 -> 41.8 mm
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Other:
- board text added: "+"
- board text added: "+ / VBUS / RED"
- board text added: "-"
- board text added: "- / GND / BLK"
- board text added: "- GND"
- board text added: "0"
- board text added: "1"
- board text added: "10"
- board text added: "11"
- board text added: "18 AWG max."
- board text added: "2"
- board text added: "2x 62Ω"
- board text added: "3"
- board text added: "4"
- board text added: "5"
- board text added: "5-26V DC"
- board text added: "500 mA total max."
- board text added: "6"
- board text added: "6A max. circuit"
- board text added: "7"
- board text added: "8"
- board text added: "9"
- board text added: "<TXD"
- board text added: ">RXD"
- board text added: "A"
- board text added: "AUX"
- board text added: "B"
- board text added: "CAN HIGH / YEL"
- board text added: "CAN LOW / GRN"
- board text added: "CANAL:"
- board text added: "COMMUNICATION"
- board text added: "CTRL"
- board text added: "FAN"
- board text added: "GND"
- board text added: "Hugo Boyce 2022-06-14 Rev.A1"
- board text added: "Instructions CANbus: - Utiliser une paire de fils torsadés. - S'assurer qu'une résistance de terminaison de 120Ω soit présente à chacune des 2 extrémités du bus. - Un ohmmètre devrait mesurer 60Ω entre les 2 fils."
- board text added: "Module d'Acquisition CANbus"
- board text added: "N"
- board text added: "NTC 10KΩ"
- board text added: "P"
- board text added: "PROG"
- board text added: "TACH"
- board text added: "TERM"
- board text added: "VOLTAGE"
- board text removed: "Check programmer mechanical fit!"
