File: CAN-Acquisition-Module_USB.kicad_sch (KiCad schematic)
At the start: 9 parts, among them J7 USB_B_Micro

Commit message: Finished power outputs
Parts:
- renumbered D9 to D11, D10 to D12, D11 to D13, D12 to D14, R23 to R24, R24 to R25, R25 to R26
Changed lines of the file:
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@@
   (symbol (lib_id "power:GND") (at 158.75 86.36 0) (unit 1)
     (in_bom yes) (on_board yes) (fields_autoplaced)
-    (property "Reference" "#PWR087" (id 0) (at 158.75 92.71 0)
+    (property "Reference" "#PWR090" (id 0) (at 158.75 92.71 0)
       (effects (font (size 1.27 1.27)) hide)
     )
@@
   (symbol (lib_id "power:+3.3V") (at 115.57 76.2 0) (unit 1)
     (in_bom yes) (on_board yes) (fields_autoplaced)
-    (property "Reference" "#PWR080" (id 0) (at 115.57 80.01 0)
+    (property "Reference" "#PWR083" (id 0) (at 115.57 80.01 0)
       (effects (font (size 1.27 1.27)) hide)
     )
@@
   (symbol (lib_id "power:GND") (at 90.17 74.93 0) (unit 1)
     (in_bom yes) (on_board yes)
-    (property "Reference" "#PWR079" (id 0) (at 90.17 81.28 0)
+    (property "Reference" "#PWR082" (id 0) (at 90.17 81.28 0)
       (effects (font (size 1.27 1.27)) hide)
     )
@@
   (symbol (lib_id "Power_Protection:CM1213A-01SO") (at 137.16 81.28 270) (unit 1)
     (in_bom yes) (on_board yes)
-    (property "Reference" "D11" (id 0) (at 139.827 80.1278 90)
+    (property "Reference" "D13" (id 0) (at 139.827 80.1278 90)
       (effects (font (size 1.27 1.27)) (justify left))
     )
@@
   (symbol (lib_id "Device:R_Small_US") (at 171.45 64.77 90) (unit 1)
     (in_bom yes) (on_board yes)
-    (property "Reference" "R24" (id 0) (at 175.26 63.5 90)
+    (property "Reference" "R25" (id 0) (at 175.26 63.5 90)
       (effects (font (size 1.27 1.27)) (justify left))
     )
@@
   (symbol (lib_id "power:+3.3V") (at 137.16 76.2 0) (unit 1)
     (in_bom yes) (on_board yes) (fields_autoplaced)
-    (property "Reference" "#PWR084" (id 0) (at 137.16 80.01 0)
+    (property "Reference" "#PWR087" (id 0) (at 137.16 80.01 0)
       (effects (font (size 1.27 1.27)) hide)
     )
@@
   (symbol (lib_id "power:+3.3V") (at 158.75 76.2 0) (unit 1)
     (in_bom yes) (on_board yes) (fields_autoplaced)
-    (property "Reference" "#PWR086" (id 0) (at 158.75 80.01 0)
+    (property "Reference" "#PWR089" (id 0) (at 158.75 80.01 0)
       (effects (font (size 1.27 1.27)) hide)
     )
@@
   (symbol (lib_id "Power_Protection:CM1213A-01SO") (at 158.75 81.28 270) (unit 1)
     (in_bom yes) (on_board yes)
-    (property "Reference" "D12" (id 0) (at 161.417 80.1278 90)
+    (property "Reference" "D14" (id 0) (at 161.417 80.1278 90)
       (effects (font (size 1.27 1.27)) (justify left))
     )
@@
   (symbol (lib_id "power:GND") (at 87.63 85.09 0) (unit 1)
     (in_bom yes) (on_board yes)
-    (property "Reference" "#PWR078" (id 0) (at 87.63 91.44 0)
+    (property "Reference" "#PWR081" (id 0) (at 87.63 91.44 0)
       (effects (font (size 1.27 1.27)) hide)
     )
@@
   (symbol (lib_id "Device:R_Small_US") (at 116.84 59.69 90) (unit 1)
     (in_bom yes) (on_board yes)
-    (property "Reference" "R23" (id 0) (at 120.65 58.42 90)
+    (property "Reference" "R24" (id 0) (at 120.65 58.42 90)
       (effects (font (size 1.27 1.27)) (justify left))
     )
@@
   (symbol (lib_id "power:+3.3V") (at 128.27 43.18 0) (unit 1)
     (in_bom yes) (on_board yes) (fields_autoplaced)
-    (property "Reference" "#PWR082" (id 0) (at 128.27 46.99 0)
+    (property "Reference" "#PWR085" (id 0) (at 128.27 46.99 0)
       (effects (font (size 1.27 1.27)) hide)
     )
@@
   (symbol (lib_id "power:GND") (at 137.16 86.36 0) (unit 1)
     (in_bom yes) (on_board yes) (fields_autoplaced)
-    (property "Reference" "#PWR085" (id 0) (at 137.16 92.71 0)
+    (property "Reference" "#PWR088" (id 0) (at 137.16 92.71 0)
       (effects (font (size 1.27 1.27)) hide)
     )
@@
   (symbol (lib_id "Power_Protection:CM1213A-01SO") (at 128.27 48.26 270) (unit 1)
     (in_bom yes) (on_board yes) (fields_autoplaced)
-    (property "Reference" "D10" (id 0) (at 130.937 47.1078 90)
+    (property "Reference" "D12" (id 0) (at 130.937 47.1078 90)
       (effects (font (size 1.27 1.27)) (justify left))
     )
@@
   (symbol (lib_id "Device:R_Small_US") (at 184.15 67.31 90) (unit 1)
     (in_bom yes) (on_board yes)
-    (property "Reference" "R25" (id 0) (at 187.96 66.04 90)
+    (property "Reference" "R26" (id 0) (at 187.96 66.04 90)
       (effects (font (size 1.27 1.27)) (justify left))
     )
@@
   (symbol (lib_id "power:GND") (at 115.57 86.36 0) (unit 1)
     (in_bom yes) (on_board yes) (fields_autoplaced)
-    (property "Reference" "#PWR081" (id 0) (at 115.57 92.71 0)
+    (property "Reference" "#PWR084" (id 0) (at 115.57 92.71 0)
       (effects (font (size 1.27 1.27)) hide)
     )
@@
   (symbol (lib_id "Power_Protection:CM1213A-01SO") (at 115.57 81.28 270) (unit 1)
     (in_bom yes) (on_board yes)
-    (property "Reference" "D9" (id 0) (at 118.237 80.1278 90)
+    (property "Reference" "D11" (id 0) (at 118.237 80.1278 90)
       (effects (font (size 1.27 1.27)) (justify left))
     )
@@
   (symbol (lib_id "power:GND") (at 128.27 53.34 0) (unit 1)
     (in_bom yes) (on_board yes) (fields_autoplaced)
-    (property "Reference" "#PWR083" (id 0) (at 128.27 59.69 0)
-      (effects (font (size 1.27 1.27)) hide)
-    )
+    (property "Reference" "#PWR086" (id 0) (at 128.27 59.69 0)
+      (effects (font (size 1.27 1.27)) hide)
+    )

Commit message: Rev. A1 release
Parts:
- renumbered R24 to R26, R25 to R27, R26 to R28
Changed lines of the file:
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@@
   (symbol (lib_id "power:GND") (at 158.75 86.36 0) (unit 1)
     (in_bom yes) (on_board yes) (fields_autoplaced)
-    (property "Reference" "#PWR091" (id 0) (at 158.75 92.71 0)
+    (property "Reference" "#PWR095" (id 0) (at 158.75 92.71 0)
       (effects (font (size 1.27 1.27)) hide)
     )
@@
   (symbol (lib_id "power:+3.3V") (at 115.57 76.2 0) (unit 1)
     (in_bom yes) (on_board yes) (fields_autoplaced)
-    (property "Reference" "#PWR084" (id 0) (at 115.57 80.01 0)
+    (property "Reference" "#PWR088" (id 0) (at 115.57 80.01 0)
       (effects (font (size 1.27 1.27)) hide)
     )
@@
   (symbol (lib_id "power:GND") (at 90.17 74.93 0) (unit 1)
     (in_bom yes) (on_board yes)
-    (property "Reference" "#PWR083" (id 0) (at 90.17 81.28 0)
+    (property "Reference" "#PWR087" (id 0) (at 90.17 81.28 0)
       (effects (font (size 1.27 1.27)) hide)
     )
@@
   (symbol (lib_id "Device:R_Small_US") (at 171.45 64.77 90) (unit 1)
     (in_bom yes) (on_board yes)
-    (property "Reference" "R25" (id 0) (at 175.26 63.5 90)
+    (property "Reference" "R27" (id 0) (at 175.26 63.5 90)
       (effects (font (size 1.27 1.27)) (justify left))
     )
@@
   (symbol (lib_id "power:+3.3V") (at 137.16 76.2 0) (unit 1)
     (in_bom yes) (on_board yes) (fields_autoplaced)
-    (property "Reference" "#PWR088" (id 0) (at 137.16 80.01 0)
+    (property "Reference" "#PWR092" (id 0) (at 137.16 80.01 0)
       (effects (font (size 1.27 1.27)) hide)
     )
@@
   (symbol (lib_id "power:+3.3V") (at 158.75 76.2 0) (unit 1)
     (in_bom yes) (on_board yes) (fields_autoplaced)
-    (property "Reference" "#PWR090" (id 0) (at 158.75 80.01 0)
+    (property "Reference" "#PWR094" (id 0) (at 158.75 80.01 0)
       (effects (font (size 1.27 1.27)) hide)
     )
@@
   (symbol (lib_id "power:GND") (at 87.63 85.09 0) (unit 1)
     (in_bom yes) (on_board yes)
-    (property "Reference" "#PWR082" (id 0) (at 87.63 91.44 0)
+    (property "Reference" "#PWR086" (id 0) (at 87.63 91.44 0)
       (effects (font (size 1.27 1.27)) hide)
     )
@@
   (symbol (lib_id "Device:R_Small_US") (at 116.84 59.69 90) (unit 1)
     (in_bom yes) (on_board yes)
-    (property "Reference" "R24" (id 0) (at 120.65 58.42 90)
+    (property "Reference" "R26" (id 0) (at 120.65 58.42 90)
       (effects (font (size 1.27 1.27)) (justify left))
     )
@@
   (symbol (lib_id "power:+3.3V") (at 128.27 43.18 0) (unit 1)
     (in_bom yes) (on_board yes) (fields_autoplaced)
-    (property "Reference" "#PWR086" (id 0) (at 128.27 46.99 0)
+    (property "Reference" "#PWR090" (id 0) (at 128.27 46.99 0)
       (effects (font (size 1.27 1.27)) hide)
     )
@@
   (symbol (lib_id "power:GND") (at 137.16 86.36 0) (unit 1)
     (in_bom yes) (on_board yes) (fields_autoplaced)
-    (property "Reference" "#PWR089" (id 0) (at 137.16 92.71 0)
+    (property "Reference" "#PWR093" (id 0) (at 137.16 92.71 0)
       (effects (font (size 1.27 1.27)) hide)
     )
@@
   (symbol (lib_id "Device:R_Small_US") (at 184.15 67.31 90) (unit 1)
     (in_bom yes) (on_board yes)
-    (property "Reference" "R26" (id 0) (at 187.96 66.04 90)
+    (property "Reference" "R28" (id 0) (at 187.96 66.04 90)
       (effects (font (size 1.27 1.27)) (justify left))
     )
@@
   (symbol (lib_id "power:GND") (at 115.57 86.36 0) (unit 1)
     (in_bom yes) (on_board yes) (fields_autoplaced)
-    (property "Reference" "#PWR085" (id 0) (at 115.57 92.71 0)
+    (property "Reference" "#PWR089" (id 0) (at 115.57 92.71 0)
       (effects (font (size 1.27 1.27)) hide)
     )
@@
   (symbol (lib_id "power:GND") (at 128.27 53.34 0) (unit 1)
     (in_bom yes) (on_board yes) (fields_autoplaced)
-    (property "Reference" "#PWR087" (id 0) (at 128.27 59.69 0)
-      (effects (font (size 1.27 1.27)) hide)
-    )
+    (property "Reference" "#PWR091" (id 0) (at 128.27 59.69 0)
+      (effects (font (size 1.27 1.27)) hide)
+    )
