File: CAN-Acquisition-Module_USB.kicad_sch (KiCad schematic)
At the start: 9 parts, among them J7 USB_B_Micro

Commit message: Added as-ordered P/Ns and regenerated Gerbers
Parts:
- D11, D12, D13, D14: Mfr. (none) -> Diodes Incorporated; P/N (none) -> D1213A-01SO-7
- L6: Mfr. (none) -> Eaton; P/N (none) -> MFBM1V1608-300-R
- R26: Mfr. (none) -> Stackpole; P/N (none) -> RMCF0603FT10K0
- R27, R28: Mfr. (none) -> Stackpole; P/N (none) -> RMCF0603FT27R0
Changed lines of the file:
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@@
+      (effects (font (size 1.27 1.27)) hide)
+    )
+    (property "Mfr." "Eaton" (id 4) (at 87.63 80.01 0)
+      (effects (font (size 1.27 1.27)) hide)
+    )
+    (property "P/N" "MFBM1V1608-300-R" (id 5) (at 87.63 80.01 0)
       (effects (font (size 1.27 1.27)) hide)
     )
@@
       (effects (font (size 1.27 1.27)) hide)
     )
+    (property "Mfr." "Diodes Incorporated" (id 4) (at 137.16 81.28 0)
+      (effects (font (size 1.27 1.27)) hide)
+    )
+    (property "P/N" "D1213A-01SO-7" (id 5) (at 137.16 81.28 0)
+      (effects (font (size 1.27 1.27)) hide)
+    )
     (pin "1")
     (pin "2")
@@
     )
     (property "Datasheet" "~" (id 3) (at 171.45 64.77 0)
+      (effects (font (size 1.27 1.27)) hide)
+    )
+    (property "Mfr." "Stackpole" (id 4) (at 171.45 64.77 0)
+      (effects (font (size 1.27 1.27)) hide)
+    )
+    (property "P/N" "RMCF0603FT27R0" (id 5) (at 171.45 64.77 0)
       (effects (font (size 1.27 1.27)) hide)
     )
@@
       (effects (font (size 1.27 1.27)) hide)
     )
+    (property "Mfr." "Diodes Incorporated" (id 4) (at 158.75 81.28 0)
+      (effects (font (size 1.27 1.27)) hide)
+    )
+    (property "P/N" "D1213A-01SO-7" (id 5) (at 158.75 81.28 0)
+      (effects (font (size 1.27 1.27)) hide)
+    )
     (pin "1")
     (pin "2")
@@
       (effects (font (size 1.27 1.27)) hide)
     )
+    (property "Mfr." "Stackpole" (id 4) (at 116.84 59.69 0)
+      (effects (font (size 1.27 1.27)) hide)
+    )
+    (property "P/N" "RMCF0603FT10K0" (id 5) (at 116.84 59.69 0)
+      (effects (font (size 1.27 1.27)) hide)
+    )
     (pin "1")
     (pin "2")
@@
       (effects (font (size 1.27 1.27)) hide)
     )
+    (property "Mfr." "Diodes Incorporated" (id 4) (at 128.27 48.26 0)
+      (effects (font (size 1.27 1.27)) hide)
+    )
+    (property "P/N" "D1213A-01SO-7" (id 5) (at 128.27 48.26 0)
+      (effects (font (size 1.27 1.27)) hide)
+    )
     (pin "1")
     (pin "2")
@@
     )
     (property "Datasheet" "~" (id 3) (at 184.15 67.31 0)
+      (effects (font (size 1.27 1.27)) hide)
+    )
+    (property "Mfr." "Stackpole" (id 4) (at 184.15 67.31 0)
+      (effects (font (size 1.27 1.27)) hide)
+    )
+    (property "P/N" "RMCF0603FT27R0" (id 5) (at 184.15 67.31 0)
       (effects (font (size 1.27 1.27)) hide)
     )
@@
       (effects (font (size 1.27 1.27)) hide)
     )
+    (property "Mfr." "Diodes Incorporated" (id 4) (at 115.57 81.28 0)
+      (effects (font (size 1.27 1.27)) hide)
+    )
+    (property "P/N" "D1213A-01SO-7" (id 5) (at 115.57 81.28 0)
+      (effects (font (size 1.27 1.27)) hide)
+    )

Commit message: BOM updated for LCSC. Still a WIP.
Parts:
- L6: LCSC (none) -> C96995
- R26, R27, R28: Tolerance (none) -> 1%
Changed lines of the file:
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@@
+      (effects (font (size 1.27 1.27)) hide)
+    )
+    (property "LCSC" "C96995" (id 6) (at 87.63 80.01 0)
       (effects (font (size 1.27 1.27)) hide)
     )
@@
     )
     (property "P/N" "RMCF0603FT27R0" (id 5) (at 171.45 64.77 0)
+      (effects (font (size 1.27 1.27)) hide)
+    )
+    (property "Tolerance" "1%" (id 6) (at 171.45 64.77 0)
       (effects (font (size 1.27 1.27)) hide)
     )
@@
       (effects (font (size 1.27 1.27)) hide)
     )
+    (property "Tolerance" "1%" (id 6) (at 116.84 59.69 0)
+      (effects (font (size 1.27 1.27)) hide)
+    )
     (pin "1")
     (pin "2")
@@
       (effects (font (size 1.27 1.27)) hide)
     )
+    (property "Tolerance" "1%" (id 6) (at 184.15 67.31 0)
+      (effects (font (size 1.27 1.27)) hide)
+    )

Commit message: BOM updated for LCSC. Still a WIP
Parts:
- D11, D12, D13, D14: LCSC (none) -> C558429
- J7: LCSC (none) -> C920231
Changed lines of the file:
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@@
+      (effects (font (size 1.27 1.27)) hide)
+    )
+    (property "LCSC" "C558429" (id 6) (at 137.16 81.28 0)
       (effects (font (size 1.27 1.27)) hide)
     )
@@
       (effects (font (size 1.27 1.27)) hide)
     )
+    (property "LCSC" "C920231" (id 6) (at 90.17 64.77 0)
+      (effects (font (size 1.27 1.27)) hide)
+    )
     (pin "1")
     (pin "2")
@@
       (effects (font (size 1.27 1.27)) hide)
     )
+    (property "LCSC" "C558429" (id 6) (at 158.75 81.28 0)
+      (effects (font (size 1.27 1.27)) hide)
+    )
     (pin "1")
     (pin "2")
@@
       (effects (font (size 1.27 1.27)) hide)
     )
+    (property "LCSC" "C558429" (id 6) (at 128.27 48.26 0)
+      (effects (font (size 1.27 1.27)) hide)
+    )
     (pin "1")
     (pin "2")
@@
       (effects (font (size 1.27 1.27)) hide)
     )
+    (property "LCSC" "C558429" (id 6) (at 115.57 81.28 0)
+      (effects (font (size 1.27 1.27)) hide)
+    )

Commit message: Created Rev B1
Replaced buck regulator S-8581AA with AP63200 because of shortage
Parts:
- D11, D12, D13, D14: LCSC C558429 -> (none); LCSC P/N (none) -> C558429; LCSC Package (none) -> SOT-23; LCSC Specs (none) -> TPCM1213A-01SO
- J7: LCSC C920231 -> (none); LCSC P/N (none) -> C920231; LCSC Package (none) -> USB; LCSC Specs (none) -> MU-106-ARWH20
- L6: LCSC C96995 -> (none); LCSC P/N (none) -> C96995; LCSC Package (none) -> 0603; LCSC Specs (none) -> UPZ1608E101-3R0TF
- R26: LCSC P/N (none) -> C98220; LCSC Package (none) -> 0603; LCSC Specs (none) -> 10K 1%
- R27, R28: LCSC P/N (none) -> C25190; LCSC Package (none) -> 0603; LCSC Specs (none) -> 27R 1%
Changed lines of the file:
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@@
       (effects (font (size 1.27 1.27)) hide)
     )
-    (property "LCSC" "C96995" (id 6) (at 87.63 80.01 0)
+    (property "LCSC" "" (id 6) (at 87.63 80.01 0)
+      (effects (font (size 1.27 1.27)) hide)
+    )
+    (property "Specs" "" (id 7) (at 87.63 80.01 0)
+      (effects (font (size 1.27 1.27)) hide)
+    )
+    (property "LCSC P/N" "C96995" (id 8) (at 87.63 80.01 0)
+      (effects (font (size 1.27 1.27)) hide)
+    )
+    (property "LCSC Specs" "UPZ1608E101-3R0TF" (id 9) (at 87.63 80.01 0)
+      (effects (font (size 1.27 1.27)) hide)
+    )
+    (property "LCSC Package" "0603" (id 10) (at 87.63 80.01 0)
       (effects (font (size 1.27 1.27)) hide)
     )
@@
       (effects (font (size 1.27 1.27)) hide)
     )
-    (property "LCSC" "C558429" (id 6) (at 137.16 81.28 0)
+    (property "LCSC" "" (id 6) (at 137.16 81.28 0)
+      (effects (font (size 1.27 1.27)) hide)
+    )
+    (property "LCSC P/N" "C558429" (id 7) (at 137.16 81.28 0)
+      (effects (font (size 1.27 1.27)) hide)
+    )
+    (property "LCSC Package" "SOT-23" (id 8) (at 137.16 81.28 0)
+      (effects (font (size 1.27 1.27)) hide)
+    )
+    (property "LCSC Specs" "TPCM1213A-01SO" (id 9) (at 137.16 81.28 0)
       (effects (font (size 1.27 1.27)) hide)
     )
@@
     )
     (property "Tolerance" "1%" (id 6) (at 171.45 64.77 0)
+      (effects (font (size 1.27 1.27)) hide)
+    )
+    (property "Specs" "" (id 7) (at 171.45 64.77 0)
+      (effects (font (size 1.27 1.27)) hide)
+    )
+    (property "LCSC" "" (id 8) (at 171.45 64.77 0)
+      (effects (font (size 1.27 1.27)) hide)
+    )
+    (property "LCSC P/N" "C25190" (id 9) (at 171.45 64.77 0)
+      (effects (font (size 1.27 1.27)) hide)
+    )
+    (property "LCSC Specs" "27R 1%" (id 10) (at 171.45 64.77 0)
+      (effects (font (size 1.27 1.27)) hide)
+    )
+    (property "LCSC Package" "0603" (id 11) (at 171.45 64.77 0)
       (effects (font (size 1.27 1.27)) hide)
     )
@@
       (effects (font (size 1.27 1.27)) hide)
     )
-    (property "LCSC" "C920231" (id 6) (at 90.17 64.77 0)
+    (property "LCSC" "" (id 6) (at 90.17 64.77 0)
+      (effects (font (size 1.27 1.27)) hide)
+    )
+    (property "Specs" "" (id 7) (at 90.17 64.77 0)
+      (effects (font (size 1.27 1.27)) hide)
+    )
+    (property "LCSC P/N" "C920231" (id 8) (at 90.17 64.77 0)
+      (effects (font (size 1.27 1.27)) hide)
+    )
+    (property "LCSC Specs" "MU-106-ARWH20" (id 9) (at 90.17 64.77 0)
+      (effects (font (size 1.27 1.27)) hide)
+    )
+    (property "LCSC Package" "USB" (id 10) (at 90.17 64.77 0)
       (effects (font (size 1.27 1.27)) hide)
     )
@@
       (effects (font (size 1.27 1.27)) hide)
     )
-    (property "LCSC" "C558429" (id 6) (at 158.75 81.28 0)
+    (property "LCSC" "" (id 6) (at 158.75 81.28 0)
+      (effects (font (size 1.27 1.27)) hide)
+    )
+    (property "LCSC P/N" "C558429" (id 7) (at 158.75 81.28 0)
+      (effects (font (size 1.27 1.27)) hide)
+    )
+    (property "LCSC Package" "SOT-23" (id 8) (at 158.75 81.28 0)
+      (effects (font (size 1.27 1.27)) hide)
+    )
+    (property "LCSC Specs" "TPCM1213A-01SO" (id 9) (at 158.75 81.28 0)
       (effects (font (size 1.27 1.27)) hide)
     )
@@
       (effects (font (size 1.27 1.27)) hide)
     )
+    (property "Specs" "" (id 7) (at 116.84 59.69 0)
+      (effects (font (size 1.27 1.27)) hide)
+    )
+    (property "LCSC" "" (id 8) (at 116.84 59.69 0)
+      (effects (font (size 1.27 1.27)) hide)
+    )
+    (property "LCSC P/N" "C98220" (id 9) (at 116.84 59.69 0)
+      (effects (font (size 1.27 1.27)) hide)
+    )
+    (property "LCSC Specs" "10K 1%" (id 10) (at 116.84 59.69 0)
+      (effects (font (size 1.27 1.27)) hide)
+    )
+    (property "LCSC Package" "0603" (id 11) (at 116.84 59.69 0)
+      (effects (font (size 1.27 1.27)) hide)
+    )
     (pin "1")
     (pin "2")
@@
       (effects (font (size 1.27 1.27)) hide)
     )
-    (property "LCSC" "C558429" (id 6) (at 128.27 48.26 0)
+    (property "LCSC" "" (id 6) (at 128.27 48.26 0)
+      (effects (font (size 1.27 1.27)) hide)
+    )
+    (property "LCSC P/N" "C558429" (id 7) (at 128.27 48.26 0)
+      (effects (font (size 1.27 1.27)) hide)
+    )
+    (property "LCSC Package" "SOT-23" (id 8) (at 128.27 48.26 0)
+      (effects (font (size 1.27 1.27)) hide)
+    )
+    (property "LCSC Specs" "TPCM1213A-01SO" (id 9) (at 128.27 48.26 0)
       (effects (font (size 1.27 1.27)) hide)
     )
@@
     )
     (property "Tolerance" "1%" (id 6) (at 184.15 67.31 0)
+      (effects (font (size 1.27 1.27)) hide)
+    )
+    (property "Specs" "" (id 7) (at 184.15 67.31 0)
+      (effects (font (size 1.27 1.27)) hide)
+    )
+    (property "LCSC" "" (id 8) (at 184.15 67.31 0)
+      (effects (font (size 1.27 1.27)) hide)
+    )
+    (property "LCSC P/N" "C25190" (id 9) (at 184.15 67.31 0)
+      (effects (font (size 1.27 1.27)) hide)
+    )
+    (property "LCSC Specs" "27R 1%" (id 10) (at 184.15 67.31 0)
+      (effects (font (size 1.27 1.27)) hide)
+    )
+    (property "LCSC Package" "0603" (id 11) (at 184.15 67.31 0)
       (effects (font (size 1.27 1.27)) hide)
     )
@@
       (effects (font (size 1.27 1.27)) hide)
     )
-    (property "LCSC" "C558429" (id 6) (at 115.57 81.28 0)
-      (effects (font (size 1.27 1.27)) hide)
-    )
+    (property "LCSC" "" (id 6) (at 115.57 81.28 0)
+      (effects (font (size 1.27 1.27)) hide)
+    )
+    (property "LCSC P/N" "C558429" (id 7) (at 115.57 81.28 0)
+      (effects (font (size 1.27 1.27)) hide)
+    )
+    (property "LCSC Package" "SOT-23" (id 8) (at 115.57 81.28 0)
+      (effects (font (size 1.27 1.27)) hide)
+    )
+    (property "LCSC Specs" "TPCM1213A-01SO" (id 9) (at 115.57 81.28 0)
+      (effects (font (size 1.27 1.27)) hide)
+    )
