File: CAN-Acqusition-Module_Sensors.kicad_sch (KiCad schematic)
At the start: 22 parts, among them U6 SCD30, U7 SHT35-DIS

Commit message: Finished power outputs
Parts:
- R48: renamed from R47; value 1.1 kΩ -> 1 kΩ
- R49: renamed from R48; value 1.1 kΩ -> 1 kΩ
- renumbered C47 to C46, C48 to C47, C49 to C48, D17 to D19, D18 to D20, R34 to R35, R35 to R36, R36 to R37, R37 to R38, R38 to R39, R39 to R40, R40 to R41, R41 to R42, R42 to R43, R43 to R44, R44 to R45, R45 to R46, R46 to R47

Commit message: Only CAN transceiver left
SPi flash should be added too
Connections:
- net +3V3: now also D19.2 (VP), D20.2 (VP)
- net GND: now also D19.3 (VN), D20.3 (VN)
Changed lines of the file:
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@@
   (junction (at 156.21 120.65) (diameter 0) (color 0 0 0 0)
   )
+  (wire (pts (xy 118.11 101.6) (xy 118.11 102.87))
+    (stroke (width 0) (type default) (color 0 0 0 0))
+  )
   (wire (pts (xy 219.71 57.15) (xy 219.71 59.69))
     (stroke (width 0) (type default) (color 0 0 0 0))
@@
     (stroke (width 0) (type default) (color 0 0 0 0))
   )
+  (wire (pts (xy 118.11 113.03) (xy 118.11 114.3))
+    (stroke (width 0) (type default) (color 0 0 0 0))
+  )
   (wire (pts (xy 86.36 130.81) (xy 87.63 130.81))
     (stroke (width 0) (type default) (color 0 0 0 0))
@@
     (stroke (width 0) (type default) (color 0 0 0 0))
   )
+  (wire (pts (xy 104.14 101.6) (xy 104.14 102.87))
+    (stroke (width 0) (type default) (color 0 0 0 0))
+  )
   (wire (pts (xy 88.9 34.29) (xy 88.9 54.61))
     (stroke (width 0) (type default) (color 0 0 0 0))
@@
     (stroke (width 0) (type default) (color 0 0 0 0))
   )
+  (wire (pts (xy 104.14 113.03) (xy 104.14 114.3))
+    (stroke (width 0) (type default) (color 0 0 0 0))
+  )

Commit message: forgor to save
Parts:
- renumbered C46 to C47, C47 to C48, C48 to C49
Changed lines of the file:
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@@
   (symbol (lib_id "power:+3.3V") (at 109.22 24.13 0) (unit 1)
     (in_bom yes) (on_board yes) (fields_autoplaced)
-    (property "Reference" "#PWR0127" (id 0) (at 109.22 27.94 0)
+    (property "Reference" "#PWR0128" (id 0) (at 109.22 27.94 0)
       (effects (font (size 1.27 1.27)) hide)
     )
@@
   (symbol (lib_id "power:GND") (at 87.63 118.11 90) (unit 1)
     (in_bom yes) (on_board yes) (fields_autoplaced)
-    (property "Reference" "#PWR0122" (id 0) (at 93.98 118.11 0)
+    (property "Reference" "#PWR0123" (id 0) (at 93.98 118.11 0)
       (effects (font (size 1.27 1.27)) hide)
     )
@@
   (symbol (lib_id "Device:C_Small") (at 55.88 121.92 0) (unit 1)
     (in_bom yes) (on_board yes)
-    (property "Reference" "C48" (id 0) (at 58.2168 120.7516 0)
+    (property "Reference" "C49" (id 0) (at 58.2168 120.7516 0)
       (effects (font (size 1.27 1.27)) (justify left))
     )
@@
   (symbol (lib_id "power:GND") (at 111.76 154.94 0) (mirror y) (unit 1)
     (in_bom yes) (on_board yes) (fields_autoplaced)
-    (property "Reference" "#PWR0130" (id 0) (at 111.76 161.29 0)
+    (property "Reference" "#PWR0131" (id 0) (at 111.76 161.29 0)
       (effects (font (size 1.27 1.27)) hide)
     )
@@
   (symbol (lib_id "power:GND") (at 76.2 43.18 0) (unit 1)
     (in_bom yes) (on_board yes) (fields_autoplaced)
-    (property "Reference" "#PWR0120" (id 0) (at 76.2 49.53 0)
+    (property "Reference" "#PWR0121" (id 0) (at 76.2 49.53 0)
       (effects (font (size 1.27 1.27)) hide)
     )
@@
   (symbol (lib_id "power:GND") (at 109.22 43.18 0) (unit 1)
     (in_bom yes) (on_board yes) (fields_autoplaced)
-    (property "Reference" "#PWR0128" (id 0) (at 109.22 49.53 0)
+    (property "Reference" "#PWR0129" (id 0) (at 109.22 49.53 0)
       (effects (font (size 1.27 1.27)) hide)
     )
@@
   (symbol (lib_id "power:+3.3V") (at 219.71 57.15 0) (unit 1)
     (in_bom yes) (on_board yes) (fields_autoplaced)
-    (property "Reference" "#PWR0134" (id 0) (at 219.71 60.96 0)
+    (property "Reference" "#PWR0135" (id 0) (at 219.71 60.96 0)
       (effects (font (size 1.27 1.27)) hide)
     )
@@
   (symbol (lib_id "power:GND") (at 46.99 128.27 0) (unit 1)
     (in_bom yes) (on_board yes) (fields_autoplaced)
-    (property "Reference" "#PWR0118" (id 0) (at 46.99 134.62 0)
+    (property "Reference" "#PWR0119" (id 0) (at 46.99 134.62 0)
       (effects (font (size 1.27 1.27)) hide)
     )
@@
   (symbol (lib_id "power:GND") (at 118.11 114.3 0) (unit 1)
     (in_bom yes) (on_board yes) (fields_autoplaced)
-    (property "Reference" "#PWR0132" (id 0) (at 118.11 120.65 0)
+    (property "Reference" "#PWR0133" (id 0) (at 118.11 120.65 0)
       (effects (font (size 1.27 1.27)) hide)
     )
@@
   (symbol (lib_id "Device:C_Small") (at 36.83 121.92 0) (unit 1)
     (in_bom yes) (on_board yes)
-    (property "Reference" "C46" (id 0) (at 39.1668 120.7516 0)
+    (property "Reference" "C47" (id 0) (at 39.1668 120.7516 0)
       (effects (font (size 1.27 1.27)) (justify left))
     )
@@
   (symbol (lib_id "Device:C_Small") (at 46.99 121.92 0) (unit 1)
     (in_bom yes) (on_board yes)
-    (property "Reference" "C47" (id 0) (at 49.3268 120.7516 0)
+    (property "Reference" "C48" (id 0) (at 49.3268 120.7516 0)
       (effects (font (size 1.27 1.27)) (justify left))
     )
@@
   (symbol (lib_id "power:GND") (at 104.14 114.3 0) (unit 1)
     (in_bom yes) (on_board yes) (fields_autoplaced)
-    (property "Reference" "#PWR0126" (id 0) (at 104.14 120.65 0)
+    (property "Reference" "#PWR0127" (id 0) (at 104.14 120.65 0)
       (effects (font (size 1.27 1.27)) hide)
     )
@@
   (symbol (lib_id "power:+3.3V") (at 111.76 135.89 0) (mirror y) (unit 1)
     (in_bom yes) (on_board yes) (fields_autoplaced)
-    (property "Reference" "#PWR0129" (id 0) (at 111.76 139.7 0)
+    (property "Reference" "#PWR0130" (id 0) (at 111.76 139.7 0)
       (effects (font (size 1.27 1.27)) hide)
     )
@@
   (symbol (lib_id "power:+3.3V") (at 104.14 101.6 0) (unit 1)
     (in_bom yes) (on_board yes) (fields_autoplaced)
-    (property "Reference" "#PWR0125" (id 0) (at 104.14 105.41 0)
+    (property "Reference" "#PWR0126" (id 0) (at 104.14 105.41 0)
       (effects (font (size 1.27 1.27)) hide)
     )
@@
   (symbol (lib_id "power:+3.3V") (at 118.11 101.6 0) (unit 1)
     (in_bom yes) (on_board yes) (fields_autoplaced)
-    (property "Reference" "#PWR0131" (id 0) (at 118.11 105.41 0)
+    (property "Reference" "#PWR0132" (id 0) (at 118.11 105.41 0)
       (effects (font (size 1.27 1.27)) hide)
     )
@@
   (symbol (lib_id "power:+3.3V") (at 76.2 24.13 0) (unit 1)
     (in_bom yes) (on_board yes) (fields_autoplaced)
-    (property "Reference" "#PWR0119" (id 0) (at 76.2 27.94 0)
+    (property "Reference" "#PWR0120" (id 0) (at 76.2 27.94 0)
       (effects (font (size 1.27 1.27)) hide)
     )
@@
   (symbol (lib_id "power:+3.3V") (at 87.63 115.57 270) (unit 1)
     (in_bom yes) (on_board yes) (fields_autoplaced)
-    (property "Reference" "#PWR0121" (id 0) (at 83.82 115.57 0)
+    (property "Reference" "#PWR0122" (id 0) (at 83.82 115.57 0)
       (effects (font (size 1.27 1.27)) hide)
     )
@@
   (symbol (lib_id "power:+3.3V") (at 88.9 24.13 0) (unit 1)
     (in_bom yes) (on_board yes) (fields_autoplaced)
-    (property "Reference" "#PWR0123" (id 0) (at 88.9 27.94 0)
+    (property "Reference" "#PWR0124" (id 0) (at 88.9 27.94 0)
       (effects (font (size 1.27 1.27)) hide)
     )
@@
   (symbol (lib_id "power:GND") (at 97.79 43.18 0) (unit 1)
     (in_bom yes) (on_board yes) (fields_autoplaced)
-    (property "Reference" "#PWR0124" (id 0) (at 97.79 49.53 0)
+    (property "Reference" "#PWR0125" (id 0) (at 97.79 49.53 0)
       (effects (font (size 1.27 1.27)) hide)
     )
@@
   (symbol (lib_id "power:+3.3V") (at 46.99 115.57 0) (unit 1)
     (in_bom yes) (on_board yes) (fields_autoplaced)
-    (property "Reference" "#PWR0117" (id 0) (at 46.99 119.38 0)
+    (property "Reference" "#PWR0118" (id 0) (at 46.99 119.38 0)
       (effects (font (size 1.27 1.27)) hide)
     )
@@
   (symbol (lib_id "power:+3.3V") (at 205.74 57.15 0) (unit 1)
     (in_bom yes) (on_board yes) (fields_autoplaced)
-    (property "Reference" "#PWR0133" (id 0) (at 205.74 60.96 0)
-      (effects (font (size 1.27 1.27)) hide)
-    )
+    (property "Reference" "#PWR0134" (id 0) (at 205.74 60.96 0)
+      (effects (font (size 1.27 1.27)) hide)
+    )

Commit message: Rev. A1 release
Parts:
- renumbered C47 to C48, C48 to C49, C49 to C50, R35 to R37, R36 to R38, R37 to R39, R38 to R40, R39 to R41, R40 to R42, R41 to R43, R42 to R44, R43 to R45, R44 to R46, R45 to R47, R46 to R48, R47 to R49, R48 to R50, R49 to R51, U6 to U7, U7 to U8
