File: CAN-Acquisition-Module.kicad_sch (KiCad schematic)
At the start: 0 parts

Commit message: PCB started
Placement well advanced
Changed lines of the file:
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@@
     (stroke (width 0) (type default) (color 0 0 0 0))
+  )
+  (label "ADC10" (at 129.54 129.54 0)
+    (effects (font (size 1.27 1.27)) (justify left bottom))
+  )
+  (label "ADC6" (at 113.03 137.16 0)
+    (effects (font (size 1.27 1.27)) (justify left bottom))
+  )
+  (label "ADC8" (at 124.46 134.62 0)
+    (effects (font (size 1.27 1.27)) (justify left bottom))
+  )
+  (label "ADC2" (at 102.87 127 0)
+    (effects (font (size 1.27 1.27)) (justify left bottom))
+  )
+  (label "ADC4" (at 107.95 132.08 0)
+    (effects (font (size 1.27 1.27)) (justify left bottom))
+  )
+  (label "ADC5" (at 110.49 134.62 0)
+    (effects (font (size 1.27 1.27)) (justify left bottom))
+  )
+  (label "ADC7" (at 115.57 139.7 0)
+    (effects (font (size 1.27 1.27)) (justify left bottom))
+  )
+  (label "ADC0" (at 97.79 121.92 0)
+    (effects (font (size 1.27 1.27)) (justify left bottom))
+  )
+  (label "ADC9" (at 127 132.08 0)
+    (effects (font (size 1.27 1.27)) (justify left bottom))
+  )
+  (label "ADC11" (at 132.08 127 0)
+    (effects (font (size 1.27 1.27)) (justify left bottom))
+  )
+  (label "ADC1" (at 100.33 124.46 0)
+    (effects (font (size 1.27 1.27)) (justify left bottom))
+  )
+  (label "ADC3" (at 105.41 129.54 0)
+    (effects (font (size 1.27 1.27)) (justify left bottom))
   )
   (sheet (at 91.44 50.8) (size 60.96 49.53) (fields_autoplaced)
@@
       (reference "#PWR058") (unit 1) (value "GND") (footprint "")
     )
-    (path "/00000000-0000-0000-0000-0000628fa103/6c024177-4eb2-4317-baa9-737627a59360"
-      (reference "#PWR059") (unit 1) (value "+1V8") (footprint "")
-    )
     (path "/00000000-0000-0000-0000-0000628fa103/00000000-0000-0000-0000-00006293b925"
       (reference "#PWR060") (unit 1) (value "GND") (footprint "")
@@
       (reference "#PWR0107") (unit 1) (value "GNDA") (footprint "")
     )
-    (path "/5f5345ca-f2d2-466f-a4ac-3c846c4226e8/39dc56cd-b644-4b00-9911-7e9e4a72be6e"
-      (reference "#PWR0108") (unit 1) (value "+3.3V") (footprint "")
-    )
-    (path "/5f5345ca-f2d2-466f-a4ac-3c846c4226e8/c9deeb0a-2b2d-4634-a0f0-57a4dfe2b754"
-      (reference "#PWR0109") (unit 1) (value "GND") (footprint "")
+    (path "/00000000-0000-0000-0000-0000628fa103/86ab31df-2e8f-432a-ae31-05629f18ef00"
+      (reference "#PWR0108") (unit 1) (value "GND") (footprint "")
+    )
+    (path "/00000000-0000-0000-0000-0000628fa103/13dad84b-9bb5-487e-8313-ed55bf3735e1"
+      (reference "#PWR0109") (unit 1) (value "+3.3V") (footprint "")
     )
     (path "/5f5345ca-f2d2-466f-a4ac-3c846c4226e8/fbb5c836-1d8f-4a79-98b1-98132a5b3174"
@@
       (reference "#PWR0176") (unit 1) (value "GNDA") (footprint "")
     )
+    (path "/8fb04998-088b-470e-9a63-5612eb9ea3de/a8530894-b37a-4f66-a4e7-e6fa6f02e8ca"
+      (reference "#PWR0177") (unit 1) (value "GNDA") (footprint "")
+    )
+    (path "/8fb04998-088b-470e-9a63-5612eb9ea3de/06b5da80-2c54-4867-a683-447ec40249ea"
+      (reference "#PWR0178") (unit 1) (value "GNDA") (footprint "")
+    )
+    (path "/8fb04998-088b-470e-9a63-5612eb9ea3de/0c93affe-9c1d-4077-b666-f221d377755e"
+      (reference "#PWR0179") (unit 1) (value "GNDA") (footprint "")
+    )
+    (path "/8fb04998-088b-470e-9a63-5612eb9ea3de/3d060349-92ed-46ce-bc0f-3c1aeef99d21"
+      (reference "#PWR0180") (unit 1) (value "GNDA") (footprint "")
+    )
+    (path "/00000000-0000-0000-0000-0000628fa103/dda72865-818d-4b3b-b854-d6d69263da6c"
+      (reference "#PWR0181") (unit 1) (value "+3.3V") (footprint "")
+    )
     (path "/00000000-0000-0000-0000-0000628fba98/00000000-0000-0000-0000-000062a4552e"
       (reference "C1") (unit 1) (value "10 uF") (footprint "Capacitor_SMD:C_0805_2012Metric")
@@
       (reference "C42") (unit 1) (value "47 uF") (footprint "Capacitor_SMD:C_1206_3216Metric")
     )
-    (path "/5f5345ca-f2d2-466f-a4ac-3c846c4226e8/7f7b9cff-1137-4a66-b751-76de8dac8bd4"
+    (path "/00000000-0000-0000-0000-0000628fa103/7d2dfb5f-dc33-4416-9abc-ab0106afcc33"
       (reference "C43") (unit 1) (value "1 uF") (footprint "Capacitor_SMD:C_0603_1608Metric")
     )
@@
       (reference "C44") (unit 1) (value "10 uF") (footprint "Capacitor_SMD:C_0805_2012Metric")
     )
-    (path "/5f5345ca-f2d2-466f-a4ac-3c846c4226e8/ff2861ee-c27c-4092-ab4b-e729fff1c6b2"
+    (path "/00000000-0000-0000-0000-0000628fa103/2589aea2-cea7-4e2b-87eb-c9d2e0fb9370"
       (reference "C45") (unit 1) (value "100 nF") (footprint "Capacitor_SMD:C_0402_1005Metric")
     )
@@
       (reference "D6") (unit 1) (value "CUS05S40") (footprint "CAN-Acquisition-Module:Toshiba_USC")
     )
+    (path "/00000000-0000-0000-0000-0000628fa103/a6728d17-eecd-4208-89cb-f7f74a736671"
+      (reference "D7") (unit 1) (value "LED_ABRG") (footprint "CAN-Acquisition-Module:LED_RGB_Wuerth-PLCC4_3.2x2.8mm_150141M173100")
+    )
     (path "/6a23b5b9-2864-4994-bd7a-8563b9182093/eed7a494-1cc8-43ba-8cd0-34f845769a10"
       (reference "D8") (unit 1) (value "PESD2CAN") (footprint "Package_TO_SOT_SMD:SOT-23")
@@
       (reference "D26") (unit 1) (value "CM1213A-01SO") (footprint "Package_TO_SOT_SMD:SOT-23")
     )
-    (path "/00000000-0000-0000-0000-0000628fa103/a6728d17-eecd-4208-89cb-f7f74a736671"
-      (reference "D?") (unit 1) (value "LED_ABRG") (footprint "CAN-Acquisition-Module:LED_RGB_Wuerth-PLCC4_3.2x2.8mm_150141M173100")
-    )
     (path "/00000000-0000-0000-0000-0000628fba98/d52911dc-6daa-4260-ab36-615528445476"
       (reference "F1") (unit 1) (value "PPTC, 50-500mA, 60V") (footprint "Fuse:Fuse_1206_3216Metric")
@@
     )
     (path "/2306ed72-7073-467c-a255-2365c3b83f36/6dfb855a-07fe-46eb-bc22-e744894aebc9"
-      (reference "J7") (unit 1) (value "USB_B_Micro") (footprint "Connector_USB:USB_Micro-B_Wuerth_614105150721_Vertical")
+      (reference "J7") (unit 1) (value "USB_B_Micro") (footprint "CAN-Acquisition-Module:GCT-USB3131-30-0230-A")
     )
     (path "/71359799-714b-4644-8db4-495310f76a1b/57a4de16-535a-46ae-af35-6b757f648165"
@@
       (reference "R74") (unit 1) (value "100 Ω") (footprint "Resistor_SMD:R_0603_1608Metric")
     )
+    (path "/8fb04998-088b-470e-9a63-5612eb9ea3de/61dedab1-3aca-4cb7-8e5d-75b430e4f4dc"
+      (reference "R75") (unit 1) (value "Ω") (footprint "Resistor_SMD:R_0603_1608Metric")
+    )
+    (path "/8fb04998-088b-470e-9a63-5612eb9ea3de/d3d9db39-6913-421b-8c0e-935c74018e9b"
+      (reference "R76") (unit 1) (value "Ω") (footprint "Resistor_SMD:R_0603_1608Metric")
+    )
+    (path "/8fb04998-088b-470e-9a63-5612eb9ea3de/cdb16de1-564a-4706-b62c-193e93a6d27e"
+      (reference "R77") (unit 1) (value "Ω") (footprint "Resistor_SMD:R_0603_1608Metric")
+    )
+    (path "/8fb04998-088b-470e-9a63-5612eb9ea3de/2346388f-2953-4c80-86bf-fab6870da8d0"
+      (reference "R78") (unit 1) (value "Ω") (footprint "Resistor_SMD:R_0603_1608Metric")
+    )
     (path "/00000000-0000-0000-0000-0000628fba98/00000000-0000-0000-0000-000062a4568c"
