File: CAN-Acquisition-Module_Analog_mV.kicad_sch (KiCad schematic)
At the start: 35 parts, among them J10 OSTVN04A150, J11 OSTVN04A150, U9 OPA4317IPWR

Commit message: Added as-ordered P/Ns and regenerated Gerbers
Parts:
- D21, D22, D23, D24: Mfr. (none) -> Diodes Incorporated; P/N (none) -> D1213A-01SO-7
- J10, J11: Mfr. (none) -> On Shore Technology
- R52, R53, R54, R55: Mfr. (none) -> Stackpole; P/N (none) -> RMCF0603FT10K0
- R60, R61, R62, R63: Mfr. (none) -> Stackpole; P/N (none) -> RMCF0603FT1K00
- R64, R65, R66, R67: Mfr. (none) -> Stackpole; P/N (none) -> RMCF0603FT2K00
- R68, R69, R70, R71: Mfr. (none) -> TE Connectivity; P/N (none) -> CRGCQ0603F47K
- U9: Mfr. (none) -> Texas Instruments; P/N (none) -> OPA4317IPWR
Changed lines of the file:
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@@
+      (effects (font (size 1.27 1.27)) hide)
+    )
+    (property "Mfr." "TE Connectivity" (id 4) (at 162.56 147.32 0)
+      (effects (font (size 1.27 1.27)) hide)
+    )
+    (property "P/N" "CRGCQ0603F47K" (id 5) (at 162.56 147.32 0)
       (effects (font (size 1.27 1.27)) hide)
     )
@@
     )
     (property "Datasheet" "https://www.ti.com/general/docs/suppproductinfo.tsp?distId=10&gotoUrl=https%3A%2F%2Fwww.ti.com%2Flit%2Fgpn%2Fopa4317" (id 3) (at 158.75 100.33 0)
+      (effects (font (size 1.27 1.27)) hide)
+    )
+    (property "Mfr." "Texas Instruments" (id 4) (at 158.75 100.33 0)
+      (effects (font (size 1.27 1.27)) hide)
+    )
+    (property "P/N" "OPA4317IPWR" (id 5) (at 158.75 100.33 0)
       (effects (font (size 1.27 1.27)) hide)
     )
@@
       (effects (font (size 1.27 1.27)) hide)
     )
+    (property "Mfr." "Stackpole" (id 4) (at 73.66 97.79 0)
+      (effects (font (size 1.27 1.27)) hide)
+    )
+    (property "P/N" "RMCF0603FT10K0" (id 5) (at 73.66 97.79 0)
+      (effects (font (size 1.27 1.27)) hide)
+    )
     (pin "1")
     (pin "2")
@@
     )
     (property "Datasheet" "~" (id 3) (at 151.13 153.67 0)
+      (effects (font (size 1.27 1.27)) hide)
+    )
+    (property "Mfr." "Stackpole" (id 4) (at 151.13 153.67 0)
+      (effects (font (size 1.27 1.27)) hide)
+    )
+    (property "P/N" "RMCF0603FT1K00" (id 5) (at 151.13 153.67 0)
       (effects (font (size 1.27 1.27)) hide)
     )
@@
       (effects (font (size 1.27 1.27)) hide)
     )
+    (property "Mfr." "On Shore Technology" (id 5) (at 46.99 25.4 0)
+      (effects (font (size 1.27 1.27)) hide)
+    )
     (pin "1")
     (pin "2")
@@
       (effects (font (size 1.27 1.27)) hide)
     )
+    (property "Mfr." "Stackpole" (id 4) (at 168.91 34.29 0)
+      (effects (font (size 1.27 1.27)) hide)
+    )
+    (property "P/N" "RMCF0603FT2K00" (id 5) (at 168.91 34.29 0)
+      (effects (font (size 1.27 1.27)) hide)
+    )
     (pin "1")
     (pin "2")
@@
     )
     (property "Datasheet" "~" (id 3) (at 176.53 69.85 0)
+      (effects (font (size 1.27 1.27)) hide)
+    )
+    (property "Mfr." "TE Connectivity" (id 4) (at 176.53 69.85 0)
+      (effects (font (size 1.27 1.27)) hide)
+    )
+    (property "P/N" "CRGCQ0603F47K" (id 5) (at 176.53 69.85 0)
       (effects (font (size 1.27 1.27)) hide)
     )
@@
       (effects (font (size 1.27 1.27)) hide)
     )
+    (property "Mfr." "Stackpole" (id 4) (at 73.66 102.87 0)
+      (effects (font (size 1.27 1.27)) hide)
+    )
+    (property "P/N" "RMCF0603FT10K0" (id 5) (at 73.66 102.87 0)
+      (effects (font (size 1.27 1.27)) hide)
+    )
     (pin "1")
     (pin "2")
@@
       (effects (font (size 1.27 1.27)) hide)
     )
+    (property "Mfr." "Stackpole" (id 4) (at 87.63 22.86 0)
+      (effects (font (size 1.27 1.27)) hide)
+    )
+    (property "P/N" "RMCF0603FT10K0" (id 5) (at 87.63 22.86 0)
+      (effects (font (size 1.27 1.27)) hide)
+    )
     (pin "1")
     (pin "2")
@@
     )
     (property "Datasheet" "~" (id 3) (at 154.94 147.32 0)
+      (effects (font (size 1.27 1.27)) hide)
+    )
+    (property "Mfr." "Stackpole" (id 4) (at 154.94 147.32 0)
+      (effects (font (size 1.27 1.27)) hide)
+    )
+    (property "P/N" "RMCF0603FT2K00" (id 5) (at 154.94 147.32 0)
       (effects (font (size 1.27 1.27)) hide)
     )
@@
       (effects (font (size 1.27 1.27)) hide)
     )
+    (property "Mfr." "Diodes Incorporated" (id 4) (at 68.58 40.64 0)
+      (effects (font (size 1.27 1.27)) hide)
+    )
+    (property "P/N" "D1213A-01SO-7" (id 5) (at 68.58 40.64 0)
+      (effects (font (size 1.27 1.27)) hide)
+    )
     (pin "1")
     (pin "2")
@@
       (effects (font (size 1.27 1.27)) hide)
     )
+    (property "Mfr." "Diodes Incorporated" (id 4) (at 67.31 115.57 0)
+      (effects (font (size 1.27 1.27)) hide)
+    )
+    (property "P/N" "D1213A-01SO-7" (id 5) (at 67.31 115.57 0)
+      (effects (font (size 1.27 1.27)) hide)
+    )
     (pin "1")
     (pin "2")
@@
       (effects (font (size 1.27 1.27)) hide)
     )
+    (property "Mfr." "Diodes Incorporated" (id 4) (at 54.61 115.57 0)
+      (effects (font (size 1.27 1.27)) hide)
+    )
+    (property "P/N" "D1213A-01SO-7" (id 5) (at 54.61 115.57 0)
+      (effects (font (size 1.27 1.27)) hide)
+    )
     (pin "1")
     (pin "2")
@@
     )
     (property "Datasheet" "~" (id 3) (at 154.94 109.22 0)
+      (effects (font (size 1.27 1.27)) hide)
+    )
+    (property "Mfr." "Stackpole" (id 4) (at 154.94 109.22 0)
+      (effects (font (size 1.27 1.27)) hide)
+    )
+    (property "P/N" "RMCF0603FT2K00" (id 5) (at 154.94 109.22 0)
       (effects (font (size 1.27 1.27)) hide)
     )
@@
     )
     (property "Datasheet" "https://www.ti.com/general/docs/suppproductinfo.tsp?distId=10&gotoUrl=https%3A%2F%2Fwww.ti.com%2Flit%2Fgpn%2Fopa4317" (id 3) (at 172.72 25.4 0)
+      (effects (font (size 1.27 1.27)) hide)
+    )
+    (property "Mfr." "Texas Instruments" (id 4) (at 172.72 25.4 0)
+      (effects (font (size 1.27 1.27)) hide)
+    )
+    (property "P/N" "OPA4317IPWR" (id 5) (at 172.72 25.4 0)
       (effects (font (size 1.27 1.27)) hide)
     )
@@
       (effects (font (size 1.27 1.27)) hide)
     )
+    (property "Mfr." "TE Connectivity" (id 4) (at 176.53 34.29 0)
+      (effects (font (size 1.27 1.27)) hide)
+    )
+    (property "P/N" "CRGCQ0603F47K" (id 5) (at 176.53 34.29 0)
+      (effects (font (size 1.27 1.27)) hide)
+    )
     (pin "1")
     (pin "2")
@@
       (effects (font (size 1.27 1.27)) hide)
     )
+    (property "Mfr." "On Shore Technology" (id 5) (at 33.02 100.33 0)
+      (effects (font (size 1.27 1.27)) hide)
+    )
     (pin "1")
     (pin "2")
@@
     )
     (property "Datasheet" "https://www.ti.com/general/docs/suppproductinfo.tsp?distId=10&gotoUrl=https%3A%2F%2Fwww.ti.com%2Flit%2Fgpn%2Fopa4317" (id 3) (at 172.72 60.96 0)
+      (effects (font (size 1.27 1.27)) hide)
+    )
+    (property "Mfr." "Texas Instruments" (id 4) (at 172.72 60.96 0)
+      (effects (font (size 1.27 1.27)) hide)
+    )
+    (property "P/N" "OPA4317IPWR" (id 5) (at 172.72 60.96 0)
       (effects (font (size 1.27 1.27)) hide)
     )
@@
       (effects (font (size 1.27 1.27)) hide)
     )
+    (property "Mfr." "Stackpole" (id 4) (at 151.13 115.57 0)
+      (effects (font (size 1.27 1.27)) hide)
+    )
+    (property "P/N" "RMCF0603FT1K00" (id 5) (at 151.13 115.57 0)
+      (effects (font (size 1.27 1.27)) hide)
+    )
     (pin "1")
     (pin "2")
@@
       (effects (font (size 1.27 1.27)) hide)
     )
+    (property "Mfr." "Stackpole" (id 4) (at 165.1 39.37 0)
+      (effects (font (size 1.27 1.27)) hide)
+    )
+    (property "P/N" "RMCF0603FT1K00" (id 5) (at 165.1 39.37 0)
+      (effects (font (size 1.27 1.27)) hide)
+    )
     (pin "1")
     (pin "2")
@@
     )
     (property "Datasheet" "~" (id 3) (at 168.91 69.85 0)
+      (effects (font (size 1.27 1.27)) hide)
+    )
+    (property "Mfr." "Stackpole" (id 4) (at 168.91 69.85 0)
+      (effects (font (size 1.27 1.27)) hide)
+    )
+    (property "P/N" "RMCF0603FT2K00" (id 5) (at 168.91 69.85 0)
       (effects (font (size 1.27 1.27)) hide)
     )
@@
       (effects (font (size 1.27 1.27)) hide)
     )
+    (property "Mfr." "Stackpole" (id 4) (at 87.63 27.94 0)
+      (effects (font (size 1.27 1.27)) hide)
+    )
+    (property "P/N" "RMCF0603FT10K0" (id 5) (at 87.63 27.94 0)
+      (effects (font (size 1.27 1.27)) hide)
+    )
     (pin "1")
     (pin "2")
@@
       (effects (font (size 1.27 1.27)) hide)
     )
+    (property "Mfr." "TE Connectivity" (id 4) (at 163.83 109.22 0)
+      (effects (font (size 1.27 1.27)) hide)
+    )
+    (property "P/N" "CRGCQ0603F47K" (id 5) (at 163.83 109.22 0)
+      (effects (font (size 1.27 1.27)) hide)
+    )
     (pin "1")
     (pin "2")
@@
       (effects (font (size 1.27 1.27)) hide)
     )
+    (property "Mfr." "Stackpole" (id 4) (at 165.1 76.2 0)
+      (effects (font (size 1.27 1.27)) hide)
+    )
+    (property "P/N" "RMCF0603FT1K00" (id 5) (at 165.1 76.2 0)
+      (effects (font (size 1.27 1.27)) hide)
+    )
     (pin "1")
     (pin "2")
@@
     )
     (property "Datasheet" "https://www.ti.com/general/docs/suppproductinfo.tsp?distId=10&gotoUrl=https%3A%2F%2Fwww.ti.com%2Flit%2Fgpn%2Fopa4317" (id 3) (at 52.07 173.99 0)
+      (effects (font (size 1.27 1.27)) hide)
+    )
+    (property "Mfr." "Texas Instruments" (id 4) (at 52.07 173.99 0)
+      (effects (font (size 1.27 1.27)) hide)
+    )
+    (property "P/N" "OPA4317IPWR" (id 5) (at 52.07 173.99 0)
       (effects (font (size 1.27 1.27)) hide)
     )
@@
       (effects (font (size 1.27 1.27)) hide)
     )
+    (property "Mfr." "Texas Instruments" (id 4) (at 158.75 138.43 0)
+      (effects (font (size 1.27 1.27)) hide)
+    )
+    (property "P/N" "OPA4317IPWR" (id 5) (at 158.75 138.43 0)
+      (effects (font (size 1.27 1.27)) hide)
+    )
     (pin "1")
     (pin "2")
@@
       (effects (font (size 1.27 1.27)) hide)
     )
+    (property "Mfr." "Diodes Incorporated" (id 4) (at 81.28 40.64 0)
+      (effects (font (size 1.27 1.27)) hide)
+    )
+    (property "P/N" "D1213A-01SO-7" (id 5) (at 81.28 40.64 0)
+      (effects (font (size 1.27 1.27)) hide)
+    )
