File: CAN-Acquisition-Module_Analog_mV.kicad_sch (KiCad schematic)
At the start: 35 parts, among them J10 OSTVN04A150, J11 OSTVN04A150, U9 OPA4317IPWR

Commit message: BOM updated for LCSC. Still a WIP.
Parts:
- J10, J11: LCSC (none) -> C708735; Mfr. On Shore Technology -> On-Shore
- R52, R53, R54, R55, R60, R61, R62, R63, R64, R65, R66, R67, R68, R69, R70, R71: Tolerance (none) -> 1%
- R56, R57, R58, R59: LCSC (none) -> DNP
- U9: LCSC (none) -> C783605
Changed lines of the file:
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@@
+      (effects (font (size 1.27 1.27)) hide)
+    )
+    (property "Tolerance" "1%" (id 6) (at 162.56 147.32 0)
       (effects (font (size 1.27 1.27)) hide)
     )
@@
     )
     (property "Do Not Place" "DNP" (id 4) (at 132.08 41.91 0))
+    (property "LCSC" "DNP" (id 5) (at 128.27 38.1 0)
+      (effects (font (size 1.27 1.27)) hide)
+    )
     (pin "1")
     (pin "2")
@@
     )
     (property "P/N" "OPA4317IPWR" (id 5) (at 158.75 100.33 0)
+      (effects (font (size 1.27 1.27)) hide)
+    )
+    (property "LCSC" "C783605" (id 6) (at 158.75 100.33 0)
       (effects (font (size 1.27 1.27)) hide)
     )
@@
       (effects (font (size 1.27 1.27)) hide)
     )
+    (property "Tolerance" "1%" (id 6) (at 73.66 97.79 0)
+      (effects (font (size 1.27 1.27)) hide)
+    )
     (pin "1")
     (pin "2")
@@
     )
     (property "P/N" "RMCF0603FT1K00" (id 5) (at 151.13 153.67 0)
+      (effects (font (size 1.27 1.27)) hide)
+    )
+    (property "Tolerance" "1%" (id 6) (at 151.13 153.67 0)
       (effects (font (size 1.27 1.27)) hide)
     )
@@
     )
     (property "Do Not Place" "DNP" (id 4) (at 91.44 116.84 0))
+    (property "LCSC" "DNP" (id 5) (at 87.63 113.03 0)
+      (effects (font (size 1.27 1.27)) hide)
+    )
     (pin "1")
     (pin "2")
@@
       (effects (font (size 1.27 1.27)) hide)
     )
-    (property "Mfr." "On Shore Technology" (id 5) (at 46.99 25.4 0)
+    (property "Mfr." "On-Shore" (id 5) (at 46.99 25.4 0)
+      (effects (font (size 1.27 1.27)) hide)
+    )
+    (property "LCSC" "C708735" (id 6) (at 46.99 25.4 0)
       (effects (font (size 1.27 1.27)) hide)
     )
@@
       (effects (font (size 1.27 1.27)) hide)
     )
+    (property "Tolerance" "1%" (id 6) (at 168.91 34.29 0)
+      (effects (font (size 1.27 1.27)) hide)
+    )
     (pin "1")
     (pin "2")
@@
     )
     (property "P/N" "CRGCQ0603F47K" (id 5) (at 176.53 69.85 0)
+      (effects (font (size 1.27 1.27)) hide)
+    )
+    (property "Tolerance" "1%" (id 6) (at 176.53 69.85 0)
       (effects (font (size 1.27 1.27)) hide)
     )
@@
       (effects (font (size 1.27 1.27)) hide)
     )
+    (property "Tolerance" "1%" (id 6) (at 73.66 102.87 0)
+      (effects (font (size 1.27 1.27)) hide)
+    )
     (pin "1")
     (pin "2")
@@
       (effects (font (size 1.27 1.27)) hide)
     )
+    (property "Tolerance" "1%" (id 6) (at 87.63 22.86 0)
+      (effects (font (size 1.27 1.27)) hide)
+    )
     (pin "1")
     (pin "2")
@@
     )
     (property "P/N" "RMCF0603FT2K00" (id 5) (at 154.94 147.32 0)
+      (effects (font (size 1.27 1.27)) hide)
+    )
+    (property "Tolerance" "1%" (id 6) (at 154.94 147.32 0)
       (effects (font (size 1.27 1.27)) hide)
     )
@@
     )
     (property "P/N" "RMCF0603FT2K00" (id 5) (at 154.94 109.22 0)
+      (effects (font (size 1.27 1.27)) hide)
+    )
+    (property "Tolerance" "1%" (id 6) (at 154.94 109.22 0)
       (effects (font (size 1.27 1.27)) hide)
     )
@@
     )
     (property "P/N" "OPA4317IPWR" (id 5) (at 172.72 25.4 0)
+      (effects (font (size 1.27 1.27)) hide)
+    )
+    (property "LCSC" "C783605" (id 6) (at 172.72 25.4 0)
       (effects (font (size 1.27 1.27)) hide)
     )
@@
       (effects (font (size 1.27 1.27)) hide)
     )
+    (property "Tolerance" "1%" (id 6) (at 176.53 34.29 0)
+      (effects (font (size 1.27 1.27)) hide)
+    )
     (pin "1")
     (pin "2")
@@
       (effects (font (size 1.27 1.27)) hide)
     )
-    (property "Mfr." "On Shore Technology" (id 5) (at 33.02 100.33 0)
+    (property "Mfr." "On-Shore" (id 5) (at 33.02 100.33 0)
+      (effects (font (size 1.27 1.27)) hide)
+    )
+    (property "LCSC" "C708735" (id 6) (at 33.02 100.33 0)
       (effects (font (size 1.27 1.27)) hide)
     )
@@
     )
     (property "P/N" "OPA4317IPWR" (id 5) (at 172.72 60.96 0)
+      (effects (font (size 1.27 1.27)) hide)
+    )
+    (property "LCSC" "C783605" (id 6) (at 172.72 60.96 0)
       (effects (font (size 1.27 1.27)) hide)
     )
@@
       (effects (font (size 1.27 1.27)) hide)
     )
+    (property "Tolerance" "1%" (id 6) (at 151.13 115.57 0)
+      (effects (font (size 1.27 1.27)) hide)
+    )
     (pin "1")
     (pin "2")
@@
       (effects (font (size 1.27 1.27)) hide)
     )
+    (property "Tolerance" "1%" (id 6) (at 165.1 39.37 0)
+      (effects (font (size 1.27 1.27)) hide)
+    )
     (pin "1")
     (pin "2")
@@
     )
     (property "P/N" "RMCF0603FT2K00" (id 5) (at 168.91 69.85 0)
+      (effects (font (size 1.27 1.27)) hide)
+    )
+    (property "Tolerance" "1%" (id 6) (at 168.91 69.85 0)
       (effects (font (size 1.27 1.27)) hide)
     )
@@
       (effects (font (size 1.27 1.27)) hide)
     )
+    (property "Tolerance" "1%" (id 6) (at 87.63 27.94 0)
+      (effects (font (size 1.27 1.27)) hide)
+    )
     (pin "1")
     (pin "2")
@@
     )
     (property "Do Not Place" "DNP" (id 4) (at 116.84 116.84 0))
+    (property "LCSC" "DNP" (id 5) (at 113.03 113.03 0)
+      (effects (font (size 1.27 1.27)) hide)
+    )
     (pin "1")
     (pin "2")
@@
     )
     (property "Do Not Place" "DNP" (id 4) (at 105.41 41.91 0))
+    (property "LCSC" "DNP" (id 5) (at 101.6 38.1 0)
+      (effects (font (size 1.27 1.27)) hide)
+    )
     (pin "1")
     (pin "2")
@@
       (effects (font (size 1.27 1.27)) hide)
     )
+    (property "Tolerance" "1%" (id 6) (at 163.83 109.22 0)
+      (effects (font (size 1.27 1.27)) hide)
+    )
     (pin "1")
     (pin "2")
@@
       (effects (font (size 1.27 1.27)) hide)
     )
+    (property "Tolerance" "1%" (id 6) (at 165.1 76.2 0)
+      (effects (font (size 1.27 1.27)) hide)
+    )
     (pin "1")
     (pin "2")
@@
     )
     (property "P/N" "OPA4317IPWR" (id 5) (at 52.07 173.99 0)
+      (effects (font (size 1.27 1.27)) hide)
+    )
+    (property "LCSC" "C783605" (id 6) (at 52.07 173.99 0)
       (effects (font (size 1.27 1.27)) hide)
     )
@@
       (effects (font (size 1.27 1.27)) hide)
     )
+    (property "LCSC" "C783605" (id 6) (at 158.75 138.43 0)
+      (effects (font (size 1.27 1.27)) hide)
+    )

Commit message: BOM updated for LCSC. Still a WIP
Parts:
- D21, D22, D23, D24: LCSC (none) -> C558429
Changed lines of the file:
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@@
+      (effects (font (size 1.27 1.27)) hide)
+    )
+    (property "LCSC" "C558429" (id 6) (at 68.58 40.64 0)
       (effects (font (size 1.27 1.27)) hide)
     )
@@
       (effects (font (size 1.27 1.27)) hide)
     )
+    (property "LCSC" "C558429" (id 6) (at 67.31 115.57 0)
+      (effects (font (size 1.27 1.27)) hide)
+    )
     (pin "1")
     (pin "2")
@@
     )
     (property "P/N" "D1213A-01SO-7" (id 5) (at 54.61 115.57 0)
+      (effects (font (size 1.27 1.27)) hide)
+    )
+    (property "LCSC" "C558429" (id 6) (at 54.61 115.57 0)
       (effects (font (size 1.27 1.27)) hide)
     )
@@
       (effects (font (size 1.27 1.27)) hide)
     )
+    (property "LCSC" "C558429" (id 6) (at 81.28 40.64 0)
+      (effects (font (size 1.27 1.27)) hide)
+    )

Commit message: Created Rev B1
Replaced buck regulator S-8581AA with AP63200 because of shortage
Parts:
- C51, C55, C56, C57, C58: LCSC P/N (none) -> C386079; LCSC Package (none) -> 0603; LCSC Specs (none) -> 1uF X7R 25V
- C52, C53, C54: LCSC P/N (none) -> C77014; LCSC Package (none) -> 0402; LCSC Specs (none) -> 100nF X7R 16V
- D21, D22, D23, D24: LCSC C558429 -> (none); LCSC P/N (none) -> C558429; LCSC Package (none) -> SOT-23; LCSC Specs (none) -> TPCM1213A-01SO
- J10, J11: LCSC C708735 -> (none); LCSC P/N (none) -> C708735; LCSC Package (none) -> 1x4 P=2.54mm; LCSC Specs (none) -> DG308-2.54-04P-14-00A(H)
- R52, R53, R54, R55: LCSC P/N (none) -> C98220; LCSC Package (none) -> 0603; LCSC Specs (none) -> 10K 1%
- R56, R57, R58, R59: LCSC DNP -> (none); LCSC P/N (none) -> DNP; LCSC Package (none) -> DNP; LCSC Specs (none) -> DNP
- R60, R61, R62, R63: LCSC P/N (none) -> C22548; LCSC Package (none) -> 0603; LCSC Specs (none) -> 1K 1%
- R64, R65, R66, R67: LCSC P/N (none) -> C22975; LCSC Package (none) -> 0603; LCSC Specs (none) -> 2K 1%
- R68, R69, R70, R71: LCSC P/N (none) -> C105579; LCSC Package (none) -> 0603; LCSC Specs (none) -> 47K 1%
- U9: LCSC C783605 -> (none); LCSC P/N (none) -> C783605; LCSC Package (none) -> TSSOP-14; LCSC Specs (none) -> OPA4317IPWR
