File: CAN-Acquisition-Module_Analog_0.kicad_sch (KiCad schematic)
At the start: 23 parts, among them J8 OSTVN04A150, J9 OSTVN04A150, U6 BD12734FVJ-E2

Commit message: Added as-ordered P/Ns and regenerated Gerbers
Parts:
- D15, D16, D17, D18: Mfr. (none) -> Diodes Incorporated; P/N (none) -> D1213A-01SO-7
- J8, J9: Mfr. (none) -> On Shore Technology
- R29, R30, R31, R32: Mfr. (none) -> Panasonic; P/N (none) -> ERA-6AEB622V
- R33, R34, R35, R36: Mfr. (none) -> Stackpole; P/N (none) -> RMCF0603JT100R
- U6: Mfr. (none) -> Rohm Semiconductor; P/N (none) -> BD12734FVJ-E2
Changed lines of the file:
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@@
+      (effects (font (size 1.27 1.27)) hide)
+    )
+    (property "Mfr." "Diodes Incorporated" (id 4) (at 77.47 114.3 0)
+      (effects (font (size 1.27 1.27)) hide)
+    )
+    (property "P/N" "D1213A-01SO-7" (id 5) (at 77.47 114.3 0)
       (effects (font (size 1.27 1.27)) hide)
     )
@@
     )
     (property "Tolerance" "0.1%" (id 4) (at 68.58 92.71 0))
+    (property "Mfr." "Panasonic" (id 5) (at 64.77 88.9 0)
+      (effects (font (size 1.27 1.27)) hide)
+    )
+    (property "P/N" "ERA-6AEB622V" (id 6) (at 64.77 88.9 0)
+      (effects (font (size 1.27 1.27)) hide)
+    )
     (pin "1")
     (pin "2")
@@
     )
     (property "Tolerance" "0.1%" (id 4) (at 68.58 27.94 0))
+    (property "Mfr." "Panasonic" (id 5) (at 64.77 24.13 0)
+      (effects (font (size 1.27 1.27)) hide)
+    )
+    (property "P/N" "ERA-6AEB622V" (id 6) (at 64.77 24.13 0)
+      (effects (font (size 1.27 1.27)) hide)
+    )
     (pin "1")
     (pin "2")
@@
     )
     (property "Datasheet" "http://www.onsemi.com/pub_link/Collateral/CM1213A-D.PDF" (id 3) (at 79.502 47.625 90)
+      (effects (font (size 1.27 1.27)) hide)
+    )
+    (property "Mfr." "Diodes Incorporated" (id 4) (at 77.47 49.53 0)
+      (effects (font (size 1.27 1.27)) hide)
+    )
+    (property "P/N" "D1213A-01SO-7" (id 5) (at 77.47 49.53 0)
       (effects (font (size 1.27 1.27)) hide)
     )
@@
     )
     (property "Datasheet" "https://fscdn.rohm.com/en/products/databook/datasheet/ic/amp_linear/opamp/bd12730g-e.pdf" (id 3) (at 168.91 137.16 0)
+      (effects (font (size 1.27 1.27)) hide)
+    )
+    (property "Mfr." "Rohm Semiconductor" (id 4) (at 168.91 137.16 0)
+      (effects (font (size 1.27 1.27)) hide)
+    )
+    (property "P/N" "BD12734FVJ-E2" (id 5) (at 168.91 137.16 0)
       (effects (font (size 1.27 1.27)) hide)
     )
@@
       (effects (font (size 1.27 1.27)) hide)
     )
+    (property "Mfr." "On Shore Technology" (id 5) (at 43.18 34.29 0)
+      (effects (font (size 1.27 1.27)) hide)
+    )
     (pin "1")
     (pin "2")
@@
       (effects (font (size 1.27 1.27)) hide)
     )
+    (property "Mfr." "On Shore Technology" (id 5) (at 43.18 99.06 0)
+      (effects (font (size 1.27 1.27)) hide)
+    )
     (pin "1")
     (pin "2")
@@
     )
     (property "Datasheet" "https://fscdn.rohm.com/en/products/databook/datasheet/ic/amp_linear/opamp/bd12730g-e.pdf" (id 3) (at 52.07 173.99 0)
+      (effects (font (size 1.27 1.27)) hide)
+    )
+    (property "Mfr." "Rohm Semiconductor" (id 4) (at 52.07 173.99 0)
+      (effects (font (size 1.27 1.27)) hide)
+    )
+    (property "P/N" "BD12734FVJ-E2" (id 5) (at 52.07 173.99 0)
       (effects (font (size 1.27 1.27)) hide)
     )
@@
       (effects (font (size 1.27 1.27)) hide)
     )
+    (property "Mfr." "Rohm Semiconductor" (id 4) (at 168.91 69.85 0)
+      (effects (font (size 1.27 1.27)) hide)
+    )
+    (property "P/N" "BD12734FVJ-E2" (id 5) (at 168.91 69.85 0)
+      (effects (font (size 1.27 1.27)) hide)
+    )
     (pin "1")
     (pin "2")
@@
       (effects (font (size 1.27 1.27)) hide)
     )
+    (property "Mfr." "Stackpole" (id 4) (at 148.59 31.75 0)
+      (effects (font (size 1.27 1.27)) hide)
+    )
+    (property "P/N" "RMCF0603JT100R" (id 5) (at 148.59 31.75 0)
+      (effects (font (size 1.27 1.27)) hide)
+    )
     (pin "1")
     (pin "2")
@@
     )
     (property "Datasheet" "https://fscdn.rohm.com/en/products/databook/datasheet/ic/amp_linear/opamp/bd12730g-e.pdf" (id 3) (at 168.91 99.06 0)
+      (effects (font (size 1.27 1.27)) hide)
+    )
+    (property "Mfr." "Rohm Semiconductor" (id 4) (at 168.91 99.06 0)
+      (effects (font (size 1.27 1.27)) hide)
+    )
+    (property "P/N" "BD12734FVJ-E2" (id 5) (at 168.91 99.06 0)
       (effects (font (size 1.27 1.27)) hide)
     )
@@
       (effects (font (size 1.27 1.27)) hide)
     )
+    (property "Mfr." "Diodes Incorporated" (id 4) (at 64.77 49.53 0)
+      (effects (font (size 1.27 1.27)) hide)
+    )
+    (property "P/N" "D1213A-01SO-7" (id 5) (at 64.77 49.53 0)
+      (effects (font (size 1.27 1.27)) hide)
+    )
     (pin "1")
     (pin "2")
@@
       (effects (font (size 1.27 1.27)) hide)
     )
+    (property "Mfr." "Stackpole" (id 4) (at 153.67 96.52 0)
+      (effects (font (size 1.27 1.27)) hide)
+    )
+    (property "P/N" "RMCF0603JT100R" (id 5) (at 153.67 96.52 0)
+      (effects (font (size 1.27 1.27)) hide)
+    )
     (pin "1")
     (pin "2")
@@
       (effects (font (size 1.27 1.27)) hide)
     )
+    (property "Mfr." "Diodes Incorporated" (id 4) (at 64.77 114.3 0)
+      (effects (font (size 1.27 1.27)) hide)
+    )
+    (property "P/N" "D1213A-01SO-7" (id 5) (at 64.77 114.3 0)
+      (effects (font (size 1.27 1.27)) hide)
+    )
     (pin "1")
     (pin "2")
@@
     )
     (property "Tolerance" "0.1%" (id 4) (at 78.74 27.94 0))
+    (property "Mfr." "Panasonic" (id 5) (at 74.93 24.13 0)
+      (effects (font (size 1.27 1.27)) hide)
+    )
+    (property "P/N" "ERA-6AEB622V" (id 6) (at 74.93 24.13 0)
+      (effects (font (size 1.27 1.27)) hide)
+    )
     (pin "1")
     (pin "2")
@@
     )
     (property "Datasheet" "https://fscdn.rohm.com/en/products/databook/datasheet/ic/amp_linear/opamp/bd12730g-e.pdf" (id 3) (at 168.91 34.29 0)
+      (effects (font (size 1.27 1.27)) hide)
+    )
+    (property "Mfr." "Rohm Semiconductor" (id 4) (at 168.91 34.29 0)
+      (effects (font (size 1.27 1.27)) hide)
+    )
+    (property "P/N" "BD12734FVJ-E2" (id 5) (at 168.91 34.29 0)
       (effects (font (size 1.27 1.27)) hide)
     )
@@
     )
     (property "Tolerance" "0.1%" (id 4) (at 78.74 92.71 0))
+    (property "Mfr." "Panasonic" (id 5) (at 74.93 88.9 0)
+      (effects (font (size 1.27 1.27)) hide)
+    )
+    (property "P/N" "ERA-6AEB622V" (id 6) (at 74.93 88.9 0)
+      (effects (font (size 1.27 1.27)) hide)
+    )
     (pin "1")
     (pin "2")
@@
       (effects (font (size 1.27 1.27)) hide)
     )
+    (property "Mfr." "Stackpole" (id 4) (at 144.78 101.6 0)
+      (effects (font (size 1.27 1.27)) hide)
+    )
+    (property "P/N" "RMCF0603JT100R" (id 5) (at 144.78 101.6 0)
+      (effects (font (size 1.27 1.27)) hide)
+    )
     (pin "1")
     (pin "2")
@@
       (effects (font (size 1.27 1.27)) hide)
     )
+    (property "Mfr." "Stackpole" (id 4) (at 142.24 36.83 0)
+      (effects (font (size 1.27 1.27)) hide)
+    )
+    (property "P/N" "RMCF0603JT100R" (id 5) (at 142.24 36.83 0)
+      (effects (font (size 1.27 1.27)) hide)
+    )
