File: CAN-Acquisition-Module_CANbus.kicad_sch (KiCad schematic)
At the start: 20 parts, among them J5 OSTVN04A150, J6 OSTVN04A150, U4 SN65HVD234

Commit message: Finished power outputs
Parts:
- renumbered C32 to C31, C33 to C32, C34 to C33, C35 to C34, C36 to C35, C37 to C36, C38 to C37, D8 to D10, R14 to R15, R15 to R16, R16 to R17, R17 to R18, R18 to R19, R19 to R20, R20 to R21, R21 to R22, R22 to R23
Changed lines of the file:
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@@
   (symbol (lib_id "power:GND") (at 156.21 130.81 0) (unit 1)
     (in_bom yes) (on_board yes) (fields_autoplaced)
-    (property "Reference" "#PWR069" (id 0) (at 156.21 137.16 0)
+    (property "Reference" "#PWR072" (id 0) (at 156.21 137.16 0)
       (effects (font (size 1.27 1.27)) hide)
     )
@@
   (symbol (lib_id "Device:R_Small_US") (at 215.9 119.38 90) (unit 1)
     (in_bom yes) (on_board yes)
-    (property "Reference" "R19" (id 0) (at 220.98 118.11 90)
+    (property "Reference" "R20" (id 0) (at 220.98 118.11 90)
       (effects (font (size 1.27 1.27)) (justify left))
     )
@@
   (symbol (lib_id "Device:R_Small_US") (at 194.31 111.76 0) (unit 1)
     (in_bom yes) (on_board yes)
-    (property "Reference" "R16" (id 0) (at 195.961 110.9253 0)
+    (property "Reference" "R17" (id 0) (at 195.961 110.9253 0)
       (effects (font (size 1.27 1.27)) (justify left))
     )
@@
   (symbol (lib_id "power:+3.3V") (at 194.31 107.95 0) (unit 1)
     (in_bom yes) (on_board yes) (fields_autoplaced)
-    (property "Reference" "#PWR072" (id 0) (at 194.31 111.76 0)
+    (property "Reference" "#PWR075" (id 0) (at 194.31 111.76 0)
       (effects (font (size 1.27 1.27)) hide)
     )
@@
   (symbol (lib_id "Device:R_Small_US") (at 214.63 97.79 90) (unit 1)
     (in_bom yes) (on_board yes)
-    (property "Reference" "R18" (id 0) (at 213.7953 96.139 0)
+    (property "Reference" "R19" (id 0) (at 213.7953 96.139 0)
       (effects (font (size 1.27 1.27)) (justify left))
     )
@@
   (symbol (lib_id "power:GND") (at 173.99 92.71 0) (unit 1)
     (in_bom yes) (on_board yes)
-    (property "Reference" "#PWR071" (id 0) (at 173.99 99.06 0)
+    (property "Reference" "#PWR074" (id 0) (at 173.99 99.06 0)
       (effects (font (size 1.27 1.27)) hide)
     )
@@
   (symbol (lib_id "Device:C_Small") (at 135.89 96.52 0) (unit 1)
     (in_bom yes) (on_board yes) (fields_autoplaced)
-    (property "Reference" "C34" (id 0) (at 138.2141 95.6916 0)
+    (property "Reference" "C33" (id 0) (at 138.2141 95.6916 0)
       (effects (font (size 1.27 1.27)) (justify left))
     )
@@
   (symbol (lib_id "power:GND") (at 233.68 106.68 0) (unit 1)
     (in_bom yes) (on_board yes) (fields_autoplaced)
-    (property "Reference" "#PWR077" (id 0) (at 233.68 113.03 0)
+    (property "Reference" "#PWR080" (id 0) (at 233.68 113.03 0)
       (effects (font (size 1.27 1.27)) hide)
     )
@@
   (symbol (lib_id "Device:R_Small_US") (at 97.79 91.44 0) (unit 1)
     (in_bom yes) (on_board yes)
-    (property "Reference" "R14" (id 0) (at 99.441 90.6053 0)
+    (property "Reference" "R15" (id 0) (at 99.441 90.6053 0)
       (effects (font (size 1.27 1.27)) (justify left))
     )
@@
   (symbol (lib_id "Device:C_Small") (at 165.1 124.46 0) (unit 1)
     (in_bom yes) (on_board yes)
-    (property "Reference" "C36" (id 0) (at 167.4368 123.2916 0)
+    (property "Reference" "C35" (id 0) (at 167.4368 123.2916 0)
       (effects (font (size 1.27 1.27)) (justify left))
     )
@@
   (symbol (lib_id "power:GND") (at 41.91 71.12 0) (unit 1)
     (in_bom yes) (on_board yes) (fields_autoplaced)
-    (property "Reference" "#PWR063" (id 0) (at 41.91 77.47 0)
+    (property "Reference" "#PWR066" (id 0) (at 41.91 77.47 0)
       (effects (font (size 1.27 1.27)) hide)
     )
@@
   (symbol (lib_id "Device:C_Small") (at 156.21 124.46 0) (unit 1)
     (in_bom yes) (on_board yes)
-    (property "Reference" "C35" (id 0) (at 158.5468 123.2916 0)
+    (property "Reference" "C34" (id 0) (at 158.5468 123.2916 0)
       (effects (font (size 1.27 1.27)) (justify left))
     )
@@
   (symbol (lib_id "power:GND") (at 67.31 97.79 0) (unit 1)
     (in_bom yes) (on_board yes) (fields_autoplaced)
-    (property "Reference" "#PWR064" (id 0) (at 67.31 104.14 0)
+    (property "Reference" "#PWR067" (id 0) (at 67.31 104.14 0)
       (effects (font (size 1.27 1.27)) hide)
     )
@@
   (symbol (lib_id "Device:R_Small_US") (at 243.84 97.79 90) (unit 1)
     (in_bom yes) (on_board yes)
-    (property "Reference" "R22" (id 0) (at 247.65 96.52 90)
+    (property "Reference" "R23" (id 0) (at 247.65 96.52 90)
       (effects (font (size 1.27 1.27)) (justify left))
     )
@@
   (symbol (lib_id "Device:C_Small") (at 233.68 102.87 0) (unit 1)
     (in_bom yes) (on_board yes)
-    (property "Reference" "C38" (id 0) (at 236.0041 102.0416 0)
+    (property "Reference" "C37" (id 0) (at 236.0041 102.0416 0)
       (effects (font (size 1.27 1.27)) (justify left))
     )
@@
   (symbol (lib_id "power:+3.3V") (at 156.21 118.11 0) (unit 1)
     (in_bom yes) (on_board yes) (fields_autoplaced)
-    (property "Reference" "#PWR068" (id 0) (at 156.21 121.92 0)
+    (property "Reference" "#PWR071" (id 0) (at 156.21 121.92 0)
       (effects (font (size 1.27 1.27)) hide)
     )
@@
   (symbol (lib_id "Device:C_Small") (at 208.28 124.46 0) (unit 1)
     (in_bom yes) (on_board yes)
-    (property "Reference" "C37" (id 0) (at 210.6041 123.6316 0)
+    (property "Reference" "C36" (id 0) (at 210.6041 123.6316 0)
       (effects (font (size 1.27 1.27)) (justify left))
     )
@@
   (symbol (lib_id "Device:C_Small") (at 124.46 96.52 0) (unit 1)
     (in_bom yes) (on_board yes) (fields_autoplaced)
-    (property "Reference" "C33" (id 0) (at 126.7841 95.6916 0)
+    (property "Reference" "C32" (id 0) (at 126.7841 95.6916 0)
       (effects (font (size 1.27 1.27)) (justify left))
     )
@@
   (symbol (lib_id "power:GND") (at 101.6 110.49 0) (unit 1)
     (in_bom yes) (on_board yes) (fields_autoplaced)
-    (property "Reference" "#PWR065" (id 0) (at 101.6 116.84 0)
+    (property "Reference" "#PWR068" (id 0) (at 101.6 116.84 0)
       (effects (font (size 1.27 1.27)) hide)
     )
@@
   (symbol (lib_id "power:GND") (at 208.28 128.27 0) (unit 1)
     (in_bom yes) (on_board yes) (fields_autoplaced)
-    (property "Reference" "#PWR074" (id 0) (at 208.28 134.62 0)
+    (property "Reference" "#PWR077" (id 0) (at 208.28 134.62 0)
       (effects (font (size 1.27 1.27)) hide)
     )
@@
   (symbol (lib_id "Device:C_Small") (at 101.6 105.41 0) (unit 1)
     (in_bom yes) (on_board yes) (fields_autoplaced)
-    (property "Reference" "C32" (id 0) (at 103.9241 104.5816 0)
+    (property "Reference" "C31" (id 0) (at 103.9241 104.5816 0)
       (effects (font (size 1.27 1.27)) (justify left))
     )
@@
   (symbol (lib_id "power:GND") (at 135.89 110.49 0) (unit 1)
     (in_bom yes) (on_board yes) (fields_autoplaced)
-    (property "Reference" "#PWR067" (id 0) (at 135.89 116.84 0)
+    (property "Reference" "#PWR070" (id 0) (at 135.89 116.84 0)
       (effects (font (size 1.27 1.27)) hide)
     )
@@
   (symbol (lib_id "power:+3.3V") (at 173.99 74.93 0) (unit 1)
     (in_bom yes) (on_board yes) (fields_autoplaced)
-    (property "Reference" "#PWR070" (id 0) (at 173.99 78.74 0)
+    (property "Reference" "#PWR073" (id 0) (at 173.99 78.74 0)
       (effects (font (size 1.27 1.27)) hide)
     )
@@
   (symbol (lib_id "power:+3.3V") (at 223.52 88.9 0) (unit 1)
     (in_bom yes) (on_board yes) (fields_autoplaced)
-    (property "Reference" "#PWR075" (id 0) (at 223.52 92.71 0)
+    (property "Reference" "#PWR078" (id 0) (at 223.52 92.71 0)
       (effects (font (size 1.27 1.27)) hide)
     )
@@
   (symbol (lib_id "power:GND") (at 194.31 128.27 0) (unit 1)
     (in_bom yes) (on_board yes) (fields_autoplaced)
-    (property "Reference" "#PWR073" (id 0) (at 194.31 134.62 0)
+    (property "Reference" "#PWR076" (id 0) (at 194.31 134.62 0)
       (effects (font (size 1.27 1.27)) hide)
     )
@@
   (symbol (lib_id "Device:R_Small_US") (at 223.52 92.71 0) (unit 1)
     (in_bom yes) (on_board yes)
-    (property "Reference" "R20" (id 0) (at 225.171 91.8753 0)
+    (property "Reference" "R21" (id 0) (at 225.171 91.8753 0)
       (effects (font (size 1.27 1.27)) (justify left))
     )
@@
   (symbol (lib_id "power:GND") (at 124.46 110.49 0) (unit 1)
     (in_bom yes) (on_board yes) (fields_autoplaced)
-    (property "Reference" "#PWR066" (id 0) (at 124.46 116.84 0)
+    (property "Reference" "#PWR069" (id 0) (at 124.46 116.84 0)
       (effects (font (size 1.27 1.27)) hide)
     )
@@
   (symbol (lib_id "Power_Protection:NUP2105L") (at 67.31 92.71 0) (unit 1)
     (in_bom yes) (on_board yes) (fields_autoplaced)
-    (property "Reference" "D8" (id 0) (at 72.517 91.8753 0)
+    (property "Reference" "D10" (id 0) (at 72.517 91.8753 0)
       (effects (font (size 1.27 1.27)) (justify left))
     )
@@
   (symbol (lib_id "Device:R_Small_US") (at 223.52 101.6 0) (unit 1)
     (in_bom yes) (on_board yes)
-    (property "Reference" "R21" (id 0) (at 225.171 100.7653 0)
+    (property "Reference" "R22" (id 0) (at 225.171 100.7653 0)
       (effects (font (size 1.27 1.27)) (justify left))
     )
@@
   (symbol (lib_id "Device:R_Small_US") (at 194.31 123.19 0) (unit 1)
     (in_bom yes) (on_board yes) (fields_autoplaced)
-    (property "Reference" "R17" (id 0) (at 195.961 122.3553 0)
+    (property "Reference" "R18" (id 0) (at 195.961 122.3553 0)
       (effects (font (size 1.27 1.27)) (justify left))
     )
@@
   (symbol (lib_id "power:GND") (at 223.52 106.68 0) (unit 1)
     (in_bom yes) (on_board yes) (fields_autoplaced)
-    (property "Reference" "#PWR076" (id 0) (at 223.52 113.03 0)
+    (property "Reference" "#PWR079" (id 0) (at 223.52 113.03 0)
       (effects (font (size 1.27 1.27)) hide)
     )
@@
   (symbol (lib_id "Device:R_Small_US") (at 106.68 91.44 0) (unit 1)
     (in_bom yes) (on_board yes)
-    (property "Reference" "R15" (id 0) (at 108.331 90.6053 0)
-      (effects (font (size 1.27 1.27)) (justify left))
-    )
+    (property "Reference" "R16" (id 0) (at 108.331 90.6053 0)
+      (effects (font (size 1.27 1.27)) (justify left))
+    )

Commit message: forgor to save
Parts:
- renumbered C31 to C32, C32 to C33, C33 to C34, C34 to C35, C35 to C36, C36 to C37, C37 to C38
Changed lines of the file:
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@@
   (symbol (lib_id "power:GND") (at 156.21 130.81 0) (unit 1)
     (in_bom yes) (on_board yes) (fields_autoplaced)
-    (property "Reference" "#PWR072" (id 0) (at 156.21 137.16 0)
+    (property "Reference" "#PWR073" (id 0) (at 156.21 137.16 0)
       (effects (font (size 1.27 1.27)) hide)
     )
@@
   (symbol (lib_id "power:+3.3V") (at 194.31 107.95 0) (unit 1)
     (in_bom yes) (on_board yes) (fields_autoplaced)
-    (property "Reference" "#PWR075" (id 0) (at 194.31 111.76 0)
+    (property "Reference" "#PWR076" (id 0) (at 194.31 111.76 0)
       (effects (font (size 1.27 1.27)) hide)
     )
@@
   (symbol (lib_id "power:GND") (at 173.99 92.71 0) (unit 1)
     (in_bom yes) (on_board yes)
-    (property "Reference" "#PWR074" (id 0) (at 173.99 99.06 0)
+    (property "Reference" "#PWR075" (id 0) (at 173.99 99.06 0)
       (effects (font (size 1.27 1.27)) hide)
     )
@@
   (symbol (lib_id "Device:C_Small") (at 135.89 96.52 0) (unit 1)
     (in_bom yes) (on_board yes) (fields_autoplaced)
-    (property "Reference" "C33" (id 0) (at 138.2141 95.6916 0)
+    (property "Reference" "C34" (id 0) (at 138.2141 95.6916 0)
       (effects (font (size 1.27 1.27)) (justify left))
     )
@@
   (symbol (lib_id "power:GND") (at 233.68 106.68 0) (unit 1)
     (in_bom yes) (on_board yes) (fields_autoplaced)
-    (property "Reference" "#PWR080" (id 0) (at 233.68 113.03 0)
+    (property "Reference" "#PWR081" (id 0) (at 233.68 113.03 0)
       (effects (font (size 1.27 1.27)) hide)
     )
@@
   (symbol (lib_id "Device:C_Small") (at 165.1 124.46 0) (unit 1)
     (in_bom yes) (on_board yes)
-    (property "Reference" "C35" (id 0) (at 167.4368 123.2916 0)
+    (property "Reference" "C36" (id 0) (at 167.4368 123.2916 0)
       (effects (font (size 1.27 1.27)) (justify left))
     )
@@
   (symbol (lib_id "power:GND") (at 41.91 71.12 0) (unit 1)
     (in_bom yes) (on_board yes) (fields_autoplaced)
-    (property "Reference" "#PWR066" (id 0) (at 41.91 77.47 0)
+    (property "Reference" "#PWR067" (id 0) (at 41.91 77.47 0)
       (effects (font (size 1.27 1.27)) hide)
     )
@@
   (symbol (lib_id "Device:C_Small") (at 156.21 124.46 0) (unit 1)
     (in_bom yes) (on_board yes)
-    (property "Reference" "C34" (id 0) (at 158.5468 123.2916 0)
+    (property "Reference" "C35" (id 0) (at 158.5468 123.2916 0)
       (effects (font (size 1.27 1.27)) (justify left))
     )
@@
   (symbol (lib_id "power:GND") (at 67.31 97.79 0) (unit 1)
     (in_bom yes) (on_board yes) (fields_autoplaced)
-    (property "Reference" "#PWR067" (id 0) (at 67.31 104.14 0)
+    (property "Reference" "#PWR068" (id 0) (at 67.31 104.14 0)
       (effects (font (size 1.27 1.27)) hide)
     )
@@
   (symbol (lib_id "Device:C_Small") (at 233.68 102.87 0) (unit 1)
     (in_bom yes) (on_board yes)
-    (property "Reference" "C37" (id 0) (at 236.0041 102.0416 0)
+    (property "Reference" "C38" (id 0) (at 236.0041 102.0416 0)
       (effects (font (size 1.27 1.27)) (justify left))
     )
@@
   (symbol (lib_id "power:+3.3V") (at 156.21 118.11 0) (unit 1)
     (in_bom yes) (on_board yes) (fields_autoplaced)
-    (property "Reference" "#PWR071" (id 0) (at 156.21 121.92 0)
+    (property "Reference" "#PWR072" (id 0) (at 156.21 121.92 0)
       (effects (font (size 1.27 1.27)) hide)
     )
@@
   (symbol (lib_id "Device:C_Small") (at 208.28 124.46 0) (unit 1)
     (in_bom yes) (on_board yes)
-    (property "Reference" "C36" (id 0) (at 210.6041 123.6316 0)
+    (property "Reference" "C37" (id 0) (at 210.6041 123.6316 0)
       (effects (font (size 1.27 1.27)) (justify left))
     )
@@
   (symbol (lib_id "Device:C_Small") (at 124.46 96.52 0) (unit 1)
     (in_bom yes) (on_board yes) (fields_autoplaced)
-    (property "Reference" "C32" (id 0) (at 126.7841 95.6916 0)
+    (property "Reference" "C33" (id 0) (at 126.7841 95.6916 0)
       (effects (font (size 1.27 1.27)) (justify left))
     )
@@
   (symbol (lib_id "power:GND") (at 101.6 110.49 0) (unit 1)
     (in_bom yes) (on_board yes) (fields_autoplaced)
-    (property "Reference" "#PWR068" (id 0) (at 101.6 116.84 0)
+    (property "Reference" "#PWR069" (id 0) (at 101.6 116.84 0)
       (effects (font (size 1.27 1.27)) hide)
     )
@@
   (symbol (lib_id "power:GND") (at 208.28 128.27 0) (unit 1)
     (in_bom yes) (on_board yes) (fields_autoplaced)
-    (property "Reference" "#PWR077" (id 0) (at 208.28 134.62 0)
+    (property "Reference" "#PWR078" (id 0) (at 208.28 134.62 0)
       (effects (font (size 1.27 1.27)) hide)
     )
@@
   (symbol (lib_id "Device:C_Small") (at 101.6 105.41 0) (unit 1)
     (in_bom yes) (on_board yes) (fields_autoplaced)
-    (property "Reference" "C31" (id 0) (at 103.9241 104.5816 0)
+    (property "Reference" "C32" (id 0) (at 103.9241 104.5816 0)
       (effects (font (size 1.27 1.27)) (justify left))
     )
@@
   (symbol (lib_id "power:GND") (at 135.89 110.49 0) (unit 1)
     (in_bom yes) (on_board yes) (fields_autoplaced)
-    (property "Reference" "#PWR070" (id 0) (at 135.89 116.84 0)
+    (property "Reference" "#PWR071" (id 0) (at 135.89 116.84 0)
       (effects (font (size 1.27 1.27)) hide)
     )
@@
   (symbol (lib_id "power:+3.3V") (at 173.99 74.93 0) (unit 1)
     (in_bom yes) (on_board yes) (fields_autoplaced)
-    (property "Reference" "#PWR073" (id 0) (at 173.99 78.74 0)
+    (property "Reference" "#PWR074" (id 0) (at 173.99 78.74 0)
       (effects (font (size 1.27 1.27)) hide)
     )
@@
   (symbol (lib_id "power:+3.3V") (at 223.52 88.9 0) (unit 1)
     (in_bom yes) (on_board yes) (fields_autoplaced)
-    (property "Reference" "#PWR078" (id 0) (at 223.52 92.71 0)
+    (property "Reference" "#PWR079" (id 0) (at 223.52 92.71 0)
       (effects (font (size 1.27 1.27)) hide)
     )
@@
   (symbol (lib_id "power:GND") (at 194.31 128.27 0) (unit 1)
     (in_bom yes) (on_board yes) (fields_autoplaced)
-    (property "Reference" "#PWR076" (id 0) (at 194.31 134.62 0)
+    (property "Reference" "#PWR077" (id 0) (at 194.31 134.62 0)
       (effects (font (size 1.27 1.27)) hide)
     )
@@
   (symbol (lib_id "power:GND") (at 124.46 110.49 0) (unit 1)
     (in_bom yes) (on_board yes) (fields_autoplaced)
-    (property "Reference" "#PWR069" (id 0) (at 124.46 116.84 0)
+    (property "Reference" "#PWR070" (id 0) (at 124.46 116.84 0)
       (effects (font (size 1.27 1.27)) hide)
     )
@@
   (symbol (lib_id "power:GND") (at 223.52 106.68 0) (unit 1)
     (in_bom yes) (on_board yes) (fields_autoplaced)
-    (property "Reference" "#PWR079" (id 0) (at 223.52 113.03 0)
-      (effects (font (size 1.27 1.27)) hide)
-    )
+    (property "Reference" "#PWR080" (id 0) (at 223.52 113.03 0)
+      (effects (font (size 1.27 1.27)) hide)
+    )
