File: CAN-Acquisition-Module_CANbus.kicad_sch (KiCad schematic)
At the start: 20 parts, among them J5 OSTVN04A150, J6 OSTVN04A150, U4 SN65HVD234

Commit message: Rev. A1 release
Parts:
- renumbered C32 to C33, C33 to C34, C34 to C35, C35 to C36, C36 to C37, C37 to C38, C38 to C39, R15 to R17, R16 to R18, R17 to R19, R18 to R20, R19 to R21, R20 to R22, R21 to R23, R22 to R24, R23 to R25, U4 to U5
Changed lines of the file:
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@@
   (symbol (lib_id "power:GND") (at 156.21 130.81 0) (unit 1)
     (in_bom yes) (on_board yes) (fields_autoplaced)
-    (property "Reference" "#PWR073" (id 0) (at 156.21 137.16 0)
+    (property "Reference" "#PWR077" (id 0) (at 156.21 137.16 0)
       (effects (font (size 1.27 1.27)) hide)
     )
@@
   (symbol (lib_id "Device:R_Small_US") (at 215.9 119.38 90) (unit 1)
     (in_bom yes) (on_board yes)
-    (property "Reference" "R20" (id 0) (at 220.98 118.11 90)
+    (property "Reference" "R22" (id 0) (at 220.98 118.11 90)
       (effects (font (size 1.27 1.27)) (justify left))
     )
@@
   (symbol (lib_id "Device:R_Small_US") (at 194.31 111.76 0) (unit 1)
     (in_bom yes) (on_board yes)
-    (property "Reference" "R17" (id 0) (at 195.961 110.9253 0)
+    (property "Reference" "R19" (id 0) (at 195.961 110.9253 0)
       (effects (font (size 1.27 1.27)) (justify left))
     )
@@
   (symbol (lib_id "power:+3.3V") (at 194.31 107.95 0) (unit 1)
     (in_bom yes) (on_board yes) (fields_autoplaced)
-    (property "Reference" "#PWR076" (id 0) (at 194.31 111.76 0)
+    (property "Reference" "#PWR080" (id 0) (at 194.31 111.76 0)
       (effects (font (size 1.27 1.27)) hide)
     )
@@
   (symbol (lib_id "Device:R_Small_US") (at 214.63 97.79 90) (unit 1)
     (in_bom yes) (on_board yes)
-    (property "Reference" "R19" (id 0) (at 213.7953 96.139 0)
+    (property "Reference" "R21" (id 0) (at 213.7953 96.139 0)
       (effects (font (size 1.27 1.27)) (justify left))
     )
@@
   (symbol (lib_id "power:GND") (at 173.99 92.71 0) (unit 1)
     (in_bom yes) (on_board yes)
-    (property "Reference" "#PWR075" (id 0) (at 173.99 99.06 0)
+    (property "Reference" "#PWR079" (id 0) (at 173.99 99.06 0)
       (effects (font (size 1.27 1.27)) hide)
     )
@@
   (symbol (lib_id "Device:C_Small") (at 135.89 96.52 0) (unit 1)
     (in_bom yes) (on_board yes) (fields_autoplaced)
-    (property "Reference" "C34" (id 0) (at 138.2141 95.6916 0)
+    (property "Reference" "C35" (id 0) (at 138.2141 95.6916 0)
       (effects (font (size 1.27 1.27)) (justify left))
     )
@@
   (symbol (lib_id "power:GND") (at 233.68 106.68 0) (unit 1)
     (in_bom yes) (on_board yes) (fields_autoplaced)
-    (property "Reference" "#PWR081" (id 0) (at 233.68 113.03 0)
+    (property "Reference" "#PWR085" (id 0) (at 233.68 113.03 0)
       (effects (font (size 1.27 1.27)) hide)
     )
@@
   (symbol (lib_id "Device:R_Small_US") (at 97.79 91.44 0) (unit 1)
     (in_bom yes) (on_board yes)
-    (property "Reference" "R15" (id 0) (at 99.441 90.6053 0)
+    (property "Reference" "R17" (id 0) (at 99.441 90.6053 0)
       (effects (font (size 1.27 1.27)) (justify left))
     )
@@
   (symbol (lib_id "Device:C_Small") (at 165.1 124.46 0) (unit 1)
     (in_bom yes) (on_board yes)
-    (property "Reference" "C36" (id 0) (at 167.4368 123.2916 0)
+    (property "Reference" "C37" (id 0) (at 167.4368 123.2916 0)
       (effects (font (size 1.27 1.27)) (justify left))
     )
@@
   (symbol (lib_id "power:GND") (at 41.91 71.12 0) (unit 1)
     (in_bom yes) (on_board yes) (fields_autoplaced)
-    (property "Reference" "#PWR067" (id 0) (at 41.91 77.47 0)
+    (property "Reference" "#PWR071" (id 0) (at 41.91 77.47 0)
       (effects (font (size 1.27 1.27)) hide)
     )
@@
   (symbol (lib_id "Device:C_Small") (at 156.21 124.46 0) (unit 1)
     (in_bom yes) (on_board yes)
-    (property "Reference" "C35" (id 0) (at 158.5468 123.2916 0)
+    (property "Reference" "C36" (id 0) (at 158.5468 123.2916 0)
       (effects (font (size 1.27 1.27)) (justify left))
     )
@@
   (symbol (lib_id "power:GND") (at 67.31 97.79 0) (unit 1)
     (in_bom yes) (on_board yes) (fields_autoplaced)
-    (property "Reference" "#PWR068" (id 0) (at 67.31 104.14 0)
+    (property "Reference" "#PWR072" (id 0) (at 67.31 104.14 0)
       (effects (font (size 1.27 1.27)) hide)
     )
@@
   (symbol (lib_id "Device:R_Small_US") (at 243.84 97.79 90) (unit 1)
     (in_bom yes) (on_board yes)
-    (property "Reference" "R23" (id 0) (at 247.65 96.52 90)
+    (property "Reference" "R25" (id 0) (at 247.65 96.52 90)
       (effects (font (size 1.27 1.27)) (justify left))
     )
@@
   (symbol (lib_id "Device:C_Small") (at 233.68 102.87 0) (unit 1)
     (in_bom yes) (on_board yes)
-    (property "Reference" "C38" (id 0) (at 236.0041 102.0416 0)
+    (property "Reference" "C39" (id 0) (at 236.0041 102.0416 0)
       (effects (font (size 1.27 1.27)) (justify left))
     )
@@
   (symbol (lib_id "power:+3.3V") (at 156.21 118.11 0) (unit 1)
     (in_bom yes) (on_board yes) (fields_autoplaced)
-    (property "Reference" "#PWR072" (id 0) (at 156.21 121.92 0)
+    (property "Reference" "#PWR076" (id 0) (at 156.21 121.92 0)
       (effects (font (size 1.27 1.27)) hide)
     )
@@
   (symbol (lib_id "Device:C_Small") (at 208.28 124.46 0) (unit 1)
     (in_bom yes) (on_board yes)
-    (property "Reference" "C37" (id 0) (at 210.6041 123.6316 0)
+    (property "Reference" "C38" (id 0) (at 210.6041 123.6316 0)
       (effects (font (size 1.27 1.27)) (justify left))
     )
@@
   (symbol (lib_id "Device:C_Small") (at 124.46 96.52 0) (unit 1)
     (in_bom yes) (on_board yes) (fields_autoplaced)
-    (property "Reference" "C33" (id 0) (at 126.7841 95.6916 0)
+    (property "Reference" "C34" (id 0) (at 126.7841 95.6916 0)
       (effects (font (size 1.27 1.27)) (justify left))
     )
@@
   (symbol (lib_id "power:GND") (at 101.6 110.49 0) (unit 1)
     (in_bom yes) (on_board yes) (fields_autoplaced)
-    (property "Reference" "#PWR069" (id 0) (at 101.6 116.84 0)
+    (property "Reference" "#PWR073" (id 0) (at 101.6 116.84 0)
       (effects (font (size 1.27 1.27)) hide)
     )
@@
   (symbol (lib_id "power:GND") (at 208.28 128.27 0) (unit 1)
     (in_bom yes) (on_board yes) (fields_autoplaced)
-    (property "Reference" "#PWR078" (id 0) (at 208.28 134.62 0)
+    (property "Reference" "#PWR082" (id 0) (at 208.28 134.62 0)
       (effects (font (size 1.27 1.27)) hide)
     )
@@
   (symbol (lib_id "Interface_CAN_LIN:SN65HVD234") (at 173.99 82.55 0) (mirror y) (unit 1)
     (in_bom yes) (on_board yes) (fields_autoplaced)
-    (property "Reference" "U4" (id 0) (at 174.5106 73.7702 0)
+    (property "Reference" "U5" (id 0) (at 174.5106 73.7702 0)
       (effects (font (size 1.27 1.27)) (justify right))
     )
@@
   (symbol (lib_id "Device:C_Small") (at 101.6 105.41 0) (unit 1)
     (in_bom yes) (on_board yes) (fields_autoplaced)
-    (property "Reference" "C32" (id 0) (at 103.9241 104.5816 0)
+    (property "Reference" "C33" (id 0) (at 103.9241 104.5816 0)
       (effects (font (size 1.27 1.27)) (justify left))
     )
@@
   (symbol (lib_id "power:GND") (at 135.89 110.49 0) (unit 1)
     (in_bom yes) (on_board yes) (fields_autoplaced)
-    (property "Reference" "#PWR071" (id 0) (at 135.89 116.84 0)
+    (property "Reference" "#PWR075" (id 0) (at 135.89 116.84 0)
       (effects (font (size 1.27 1.27)) hide)
     )
@@
   (symbol (lib_id "power:+3.3V") (at 173.99 74.93 0) (unit 1)
     (in_bom yes) (on_board yes) (fields_autoplaced)
-    (property "Reference" "#PWR074" (id 0) (at 173.99 78.74 0)
+    (property "Reference" "#PWR078" (id 0) (at 173.99 78.74 0)
       (effects (font (size 1.27 1.27)) hide)
     )
@@
   (symbol (lib_id "power:+3.3V") (at 223.52 88.9 0) (unit 1)
     (in_bom yes) (on_board yes) (fields_autoplaced)
-    (property "Reference" "#PWR079" (id 0) (at 223.52 92.71 0)
+    (property "Reference" "#PWR083" (id 0) (at 223.52 92.71 0)
       (effects (font (size 1.27 1.27)) hide)
     )
@@
   (symbol (lib_id "power:GND") (at 194.31 128.27 0) (unit 1)
     (in_bom yes) (on_board yes) (fields_autoplaced)
-    (property "Reference" "#PWR077" (id 0) (at 194.31 134.62 0)
+    (property "Reference" "#PWR081" (id 0) (at 194.31 134.62 0)
       (effects (font (size 1.27 1.27)) hide)
     )
@@
   (symbol (lib_id "Device:R_Small_US") (at 223.52 92.71 0) (unit 1)
     (in_bom yes) (on_board yes)
-    (property "Reference" "R21" (id 0) (at 225.171 91.8753 0)
+    (property "Reference" "R23" (id 0) (at 225.171 91.8753 0)
       (effects (font (size 1.27 1.27)) (justify left))
     )
@@
   (symbol (lib_id "power:GND") (at 124.46 110.49 0) (unit 1)
     (in_bom yes) (on_board yes) (fields_autoplaced)
-    (property "Reference" "#PWR070" (id 0) (at 124.46 116.84 0)
+    (property "Reference" "#PWR074" (id 0) (at 124.46 116.84 0)
       (effects (font (size 1.27 1.27)) hide)
     )
@@
   (symbol (lib_id "Device:R_Small_US") (at 223.52 101.6 0) (unit 1)
     (in_bom yes) (on_board yes)
-    (property "Reference" "R22" (id 0) (at 225.171 100.7653 0)
+    (property "Reference" "R24" (id 0) (at 225.171 100.7653 0)
       (effects (font (size 1.27 1.27)) (justify left))
     )
@@
   (symbol (lib_id "Device:R_Small_US") (at 194.31 123.19 0) (unit 1)
     (in_bom yes) (on_board yes) (fields_autoplaced)
-    (property "Reference" "R18" (id 0) (at 195.961 122.3553 0)
+    (property "Reference" "R20" (id 0) (at 195.961 122.3553 0)
       (effects (font (size 1.27 1.27)) (justify left))
     )
@@
   (symbol (lib_id "power:GND") (at 223.52 106.68 0) (unit 1)
     (in_bom yes) (on_board yes) (fields_autoplaced)
-    (property "Reference" "#PWR080" (id 0) (at 223.52 113.03 0)
+    (property "Reference" "#PWR084" (id 0) (at 223.52 113.03 0)
       (effects (font (size 1.27 1.27)) hide)
     )
@@
   (symbol (lib_id "Device:R_Small_US") (at 106.68 91.44 0) (unit 1)
     (in_bom yes) (on_board yes)
-    (property "Reference" "R16" (id 0) (at 108.331 90.6053 0)
-      (effects (font (size 1.27 1.27)) (justify left))
-    )
+    (property "Reference" "R18" (id 0) (at 108.331 90.6053 0)
+      (effects (font (size 1.27 1.27)) (justify left))
+    )

Commit message: Added as-ordered P/Ns and regenerated Gerbers
Parts:
- C34, C35: Mfr. (none) -> Samsung; P/N (none) -> CL10C470JB81PNC
- D10: Mfr. (none) -> Comchip Technology; P/N (none) -> CPDT-24V
- J5, J6: Mfr. (none) -> On Shore Technology
- R20: Mfr. (none) -> Stackpole; P/N (none) -> RMCF0603FT22K0
- R25: Mfr. (none) -> Stackpole; P/N (none) -> RMCF0603FT1K00
Changed lines of the file:
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@@
+      (effects (font (size 1.27 1.27)) hide)
+    )
+    (property "Mfr." "Samsung" (id 4) (at 135.89 96.52 0)
+      (effects (font (size 1.27 1.27)) hide)
+    )
+    (property "P/N" "CL10C470JB81PNC" (id 5) (at 135.89 96.52 0)
       (effects (font (size 1.27 1.27)) hide)
     )
@@
       (effects (font (size 1.27 1.27)) hide)
     )
+    (property "Mfr." "On Shore Technology" (id 5) (at 66.04 67.31 0)
+      (effects (font (size 1.27 1.27)) hide)
+    )
     (pin "1")
     (pin "2")
@@
       (effects (font (size 1.27 1.27)) hide)
     )
+    (property "Mfr." "Stackpole" (id 4) (at 243.84 97.79 0)
+      (effects (font (size 1.27 1.27)) hide)
+    )
+    (property "P/N" "RMCF0603FT1K00" (id 5) (at 243.84 97.79 0)
+      (effects (font (size 1.27 1.27)) hide)
+    )
     (pin "1")
     (pin "2")
@@
     )
     (property "Datasheet" "~" (id 3) (at 124.46 96.52 0)
+      (effects (font (size 1.27 1.27)) hide)
+    )
+    (property "Mfr." "Samsung" (id 4) (at 124.46 96.52 0)
+      (effects (font (size 1.27 1.27)) hide)
+    )
+    (property "P/N" "CL10C470JB81PNC" (id 5) (at 124.46 96.52 0)
       (effects (font (size 1.27 1.27)) hide)
     )
@@
       (effects (font (size 1.27 1.27)) hide)
     )
+    (property "Mfr." "Comchip Technology" (id 4) (at 67.31 92.71 0)
+      (effects (font (size 1.27 1.27)) hide)
+    )
+    (property "P/N" "CPDT-24V" (id 5) (at 67.31 92.71 0)
+      (effects (font (size 1.27 1.27)) hide)
+    )
     (pin "3")
     (pin "1")
@@
       (effects (font (size 1.27 1.27)) hide)
     )
+    (property "Mfr." "On Shore Technology" (id 5) (at 36.83 64.77 0)
+      (effects (font (size 1.27 1.27)) hide)
+    )
     (pin "1")
     (pin "2")
@@
       (effects (font (size 1.27 1.27)) hide)
     )
+    (property "Mfr." "Stackpole" (id 4) (at 194.31 123.19 0)
+      (effects (font (size 1.27 1.27)) hide)
+    )
+    (property "P/N" "RMCF0603FT22K0" (id 5) (at 194.31 123.19 0)
+      (effects (font (size 1.27 1.27)) hide)
+    )

Commit message: BOM updated for LCSC. Still a WIP.
Parts:
- C33, C38, C39, R17, R18, R19, R21, R22, R23, R24: LCSC (none) -> DNP
- J5, J6: LCSC (none) -> C708735; Mfr. On Shore Technology -> On-Shore
- R20, R25: Tolerance (none) -> 1%
- U5: LCSC (none) -> C111810
Changed lines of the file:
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@@
     )
     (property "Do Not Place" "DNP" (id 4) (at 219.71 123.19 90))
+    (property "LCSC" "DNP" (id 5) (at 215.9 119.38 0)
+      (effects (font (size 1.27 1.27)) hide)
+    )
     (pin "1")
     (pin "2")
@@
     )
     (property "Do Not Place" "DNP" (id 4) (at 198.12 115.57 0))
+    (property "LCSC" "DNP" (id 5) (at 194.31 111.76 0)
+      (effects (font (size 1.27 1.27)) hide)
+    )
     (pin "1")
     (pin "2")
@@
     )
     (property "Do Not Place" "DNP" (id 4) (at 218.44 93.98 0))
+    (property "LCSC" "DNP" (id 5) (at 214.63 97.79 0)
+      (effects (font (size 1.27 1.27)) hide)
+    )
     (pin "1")
     (pin "2")
@@
     )
     (property "Do Not Place" "DNP" (id 4) (at 100.33 93.98 0))
+    (property "LCSC" "DNP" (id 5) (at 97.79 91.44 0)
+      (effects (font (size 1.27 1.27)) hide)
+    )
     (pin "1")
     (pin "2")
@@
       (effects (font (size 1.27 1.27)) hide)
     )
-    (property "Mfr." "On Shore Technology" (id 5) (at 66.04 67.31 0)
+    (property "Mfr." "On-Shore" (id 5) (at 66.04 67.31 0)
+      (effects (font (size 1.27 1.27)) hide)
+    )
+    (property "LCSC" "C708735" (id 6) (at 66.04 67.31 0)
       (effects (font (size 1.27 1.27)) hide)
     )
@@
       (effects (font (size 1.27 1.27)) hide)
     )
+    (property "Tolerance" "1%" (id 6) (at 243.84 97.79 0)
+      (effects (font (size 1.27 1.27)) hide)
+    )
     (pin "1")
     (pin "2")
@@
     )
     (property "Do Not Place" "DNP" (id 4) (at 237.49 106.68 0))
+    (property "LCSC" "DNP" (id 5) (at 233.68 102.87 0)
+      (effects (font (size 1.27 1.27)) hide)
+    )
     (pin "1")
     (pin "2")
@@
     )
     (property "Do Not Place" "DNP" (id 4) (at 213.36 128.27 0))
+    (property "LCSC" "DNP" (id 5) (at 208.28 124.46 0)
+      (effects (font (size 1.27 1.27)) hide)
+    )
     (pin "1")
     (pin "2")
@@
     )
     (property "Datasheet" "http://www.ti.com/lit/ds/symlink/sn65hvd234.pdf" (id 3) (at 176.53 72.39 0)
+      (effects (font (size 1.27 1.27)) hide)
+    )
+    (property "LCSC" "C111810" (id 4) (at 173.99 82.55 0)
       (effects (font (size 1.27 1.27)) hide)
     )
@@
       (effects (font (size 1.27 1.27)) hide)
     )
+    (property "LCSC" "DNP" (id 5) (at 101.6 105.41 0)
+      (effects (font (size 1.27 1.27)) hide)
+    )
     (pin "1")
     (pin "2")
@@
     )
     (property "Do Not Place" "DNP" (id 4) (at 227.33 96.52 0))
+    (property "LCSC" "DNP" (id 5) (at 223.52 92.71 0)
+      (effects (font (size 1.27 1.27)) hide)
+    )
     (pin "1")
     (pin "2")
@@
     )
     (property "Do Not Place" "DNP" (id 4) (at 227.33 105.41 0))
+    (property "LCSC" "DNP" (id 5) (at 223.52 101.6 0)
+      (effects (font (size 1.27 1.27)) hide)
+    )
     (pin "1")
     (pin "2")
@@
       (effects (font (size 1.27 1.27)) hide)
     )
-    (property "Mfr." "On Shore Technology" (id 5) (at 36.83 64.77 0)
+    (property "Mfr." "On-Shore" (id 5) (at 36.83 64.77 0)
+      (effects (font (size 1.27 1.27)) hide)
+    )
+    (property "LCSC" "C708735" (id 6) (at 36.83 64.77 0)
       (effects (font (size 1.27 1.27)) hide)
     )
@@
       (effects (font (size 1.27 1.27)) hide)
     )
+    (property "Tolerance" "1%" (id 6) (at 194.31 123.19 0)
+      (effects (font (size 1.27 1.27)) hide)
+    )
     (pin "1")
     (pin "2")
@@
     )
     (property "Do Not Place" "DNP" (id 4) (at 109.22 93.98 0))
-    (pin "1")
-    (pin "2")
+    (property "LCSC" "DNP" (id 5) (at 106.68 91.44 0)
+      (effects (font (size 1.27 1.27)) hide)
+    )
+    (pin "1")
+    (pin "2")

Commit message: BOM updated for LCSC. Still a WIP
Parts:
- D10: LCSC (none) -> C284078
Changed lines of the file:
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@@
+      (effects (font (size 1.27 1.27)) hide)
+    )
+    (property "LCSC" "C284078" (id 6) (at 67.31 92.71 0)
       (effects (font (size 1.27 1.27)) hide)
     )

Commit message: Added differential BOM for order (to be removed later)
Parts:
- U5: value SN65HVD234 -> SN65HVD235
Changed lines of the file:
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@@
     (stroke (width 0) (type default) (color 0 0 0 0))
   )
-  (polyline (pts (xy 203.2 137.16) (xy 240.03 137.16))
+  (polyline (pts (xy 203.2 137.16) (xy 241.3 137.16))
     (stroke (width 0) (type default) (color 0 0 0 0))
   )
@@
     (stroke (width 0) (type default) (color 0 0 0 0))
   )
-  (polyline (pts (xy 240.03 137.16) (xy 240.03 88.9))
+  (polyline (pts (xy 241.3 137.16) (xy 241.3 88.9))
     (stroke (width 0) (type default) (color 0 0 0 0))
   )
@@
     (stroke (width 0) (type default) (color 0 0 0 0))
   )
-  (polyline (pts (xy 240.03 88.9) (xy 190.5 88.9))
+  (polyline (pts (xy 241.3 88.9) (xy 190.5 88.9))
     (stroke (width 0) (type default) (color 0 0 0 0))
   )
@@
   (symbol (lib_id "Device:R_Small_US") (at 243.84 97.79 90) (unit 1)
     (in_bom yes) (on_board yes)
-    (property "Reference" "R25" (id 0) (at 247.65 96.52 90)
+    (property "Reference" "R25" (id 0) (at 248.92 96.52 90)
       (effects (font (size 1.27 1.27)) (justify left))
     )
@@
     )
     (property "Tolerance" "1%" (id 6) (at 243.84 97.79 0)
+      (effects (font (size 1.27 1.27)) hide)
+    )
+    (property "Do Not Place" "" (id 7) (at 247.65 101.6 90)
       (effects (font (size 1.27 1.27)) hide)
     )
@@
   (symbol (lib_id "Interface_CAN_LIN:SN65HVD234") (at 173.99 82.55 0) (mirror y) (unit 1)
     (in_bom yes) (on_board yes) (fields_autoplaced)
-    (property "Reference" "U5" (id 0) (at 174.5106 73.7702 0)
+    (property "Reference" "U5" (id 0) (at 173.4694 73.7702 0)
       (effects (font (size 1.27 1.27)) (justify right))
     )
-    (property "Value" "SN65HVD234" (id 1) (at 174.5106 76.3071 0)
+    (property "Value" "SN65HVD235" (id 1) (at 173.4694 76.3071 0)
       (effects (font (size 1.27 1.27)) (justify right))
     )
@@
       (effects (font (size 1.27 1.27)) hide)
     )
-    (property "Datasheet" "http://www.ti.com/lit/ds/symlink/sn65hvd234.pdf" (id 3) (at 176.53 72.39 0)
-      (effects (font (size 1.27 1.27)) hide)
-    )
+    (property "Datasheet" "http://www.ti.com/lit/ds/symlink/sn65hvd234.pdf" (id 3) (at 171.45 72.39 0)
+      (effects (font (size 1.27 1.27)) hide)
+    )
