File: CAN-Acquisition-Module_MCU.kicad_sch (KiCad schematic)
At the start: 39 parts, among them J3 Conn_01x03, J4 Conn_02x05_Odd_Even, U3 M483SGCAE, U4 SST25VF080B-50-4x-S2Ax, Y1 12 MHz

Commit message: BOM updated for LCSC. Still a WIP.
Parts:
- L4, L5: LCSC (none) -> C96995
- R10, R11, R12, R13, R14, R16: Tolerance (none) -> 1%
- R15: LCSC (none) -> DNP
- U3: LCSC (none) -> C3231235
- U4: Do Not Place (none) -> DNP; LCSC (none) -> DNP
- Y1: LCSC (none) -> C91749
Changed lines of the file:
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@@
+      (effects (font (size 1.27 1.27)) hide)
+    )
+    (property "LCSC" "C3231235" (id 6) (at 107.95 54.61 0)
       (effects (font (size 1.27 1.27)) hide)
     )
@@
       (effects (font (size 1.27 1.27)) hide)
     )
+    (property "Tolerance" "1%" (id 6) (at 270.51 45.72 0)
+      (effects (font (size 1.27 1.27)) hide)
+    )
     (pin "1")
     (pin "2")
@@
     )
     (property "P/N" "C3E-12.000-18-3030-X-R" (id 5) (at 182.88 106.68 0)
+      (effects (font (size 1.27 1.27)) hide)
+    )
+    (property "LCSC" "C91749" (id 6) (at 182.88 106.68 0)
       (effects (font (size 1.27 1.27)) hide)
     )
@@
       (effects (font (size 1.27 1.27)) hide)
     )
+    (property "LCSC" "C96995" (id 6) (at 34.29 149.86 0)
+      (effects (font (size 1.27 1.27)) hide)
+    )
     (pin "1")
     (pin "2")
@@
       (effects (font (size 1.27 1.27)) hide)
     )
+    (property "LCSC" "C96995" (id 6) (at 34.29 139.7 0)
+      (effects (font (size 1.27 1.27)) hide)
+    )
     (pin "1")
     (pin "2")
@@
       (effects (font (size 1.27 1.27)) hide)
     )
+    (property "Tolerance" "1%" (id 6) (at 55.88 71.12 0)
+      (effects (font (size 1.27 1.27)) hide)
+    )
     (pin "1")
     (pin "2")
@@
       (effects (font (size 1.27 1.27)) hide)
     )
+    (property "Tolerance" "1%" (id 6) (at 208.28 140.97 0)
+      (effects (font (size 1.27 1.27)) hide)
+    )
     (pin "1")
     (pin "2")
@@
       (effects (font (size 1.27 1.27)) hide)
     )
+    (property "Tolerance" "1%" (id 6) (at 55.88 76.2 0)
+      (effects (font (size 1.27 1.27)) hide)
+    )
     (pin "1")
     (pin "2")
@@
     )
     (property "Do Not Place" "DNP" (id 4) (at 265.43 40.005 90))
+    (property "LCSC" "DNP" (id 5) (at 265.43 41.91 0)
+      (effects (font (size 1.27 1.27)) hide)
+    )
     (pin "1")
     (pin "2")
@@
     )
     (property "Datasheet" "http://ww1.microchip.com/downloads/en/DeviceDoc/20005045C.pdf" (id 3) (at 236.22 130.81 0)
+      (effects (font (size 1.27 1.27)) hide)
+    )
+    (property "Do Not Place" "DNP" (id 4) (at 237.49 144.78 0)
+      (effects (font (size 1.27 1.27)) hide)
+    )
+    (property "LCSC" "DNP" (id 5) (at 237.49 144.78 0)
       (effects (font (size 1.27 1.27)) hide)
     )
@@
       (effects (font (size 1.27 1.27)) hide)
     )
+    (property "Tolerance" "1%" (id 6) (at 199.39 140.97 0)
+      (effects (font (size 1.27 1.27)) hide)
+    )
     (pin "1")
     (pin "2")
@@
       (effects (font (size 1.27 1.27)) hide)
     )
+    (property "Tolerance" "1%" (id 6) (at 55.88 66.04 0)
+      (effects (font (size 1.27 1.27)) hide)
+    )

Commit message: BOM updated for LCSC. Still a WIP
Parts:
- D7: Alternate P/N (none) -> MHPA3528RGBCT; LCSC (none) -> C409779
- D8, D9: LCSC (none) -> C558429
- H1, H2, H3, H4, J3: Do Not Place (none) -> DNP; LCSC (none) -> DNP
- J4: LCSC (none) -> C124387
Changed lines of the file:
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@@
+      (effects (font (size 1.27 1.27)) hide)
+    )
+    (property "LCSC" "C124387" (id 4) (at 247.65 46.99 0)
       (effects (font (size 1.27 1.27)) hide)
     )
@@
       (effects (font (size 1.27 1.27)) hide)
     )
+    (property "Do Not Place" "DNP" (id 4) (at 158.75 171.45 0)
+      (effects (font (size 1.27 1.27)) hide)
+    )
+    (property "LCSC" "DNP" (id 5) (at 158.75 171.45 0)
+      (effects (font (size 1.27 1.27)) hide)
+    )
   )
   (symbol (lib_id "Device:Crystal_GND24_Small") (at 182.88 106.68 270) (unit 1)
@@
       (effects (font (size 1.27 1.27)) hide)
     )
+    (property "LCSC" "C558429" (id 6) (at 113.03 152.4 0)
+      (effects (font (size 1.27 1.27)) hide)
+    )
     (pin "1")
     (pin "2")
@@
     )
     (property "Datasheet" "~" (id 3) (at 158.75 190.5 0)
+      (effects (font (size 1.27 1.27)) hide)
+    )
+    (property "Do Not Place" "DNP" (id 4) (at 158.75 190.5 0)
+      (effects (font (size 1.27 1.27)) hide)
+    )
+    (property "LCSC" "DNP" (id 5) (at 158.75 190.5 0)
       (effects (font (size 1.27 1.27)) hide)
     )
@@
       (effects (font (size 1.27 1.27)) hide)
     )
+    (property "Do Not Place" "DNP" (id 4) (at 158.75 177.8 0)
+      (effects (font (size 1.27 1.27)) hide)
+    )
+    (property "LCSC" "DNP" (id 5) (at 158.75 177.8 0)
+      (effects (font (size 1.27 1.27)) hide)
+    )
   )
   (symbol (lib_id "power:+1V8") (at 83.82 170.18 0) (unit 1)
@@
       (effects (font (size 1.27 1.27)) hide)
     )
+    (property "LCSC" "C558429" (id 6) (at 124.46 152.4 0)
+      (effects (font (size 1.27 1.27)) hide)
+    )
     (pin "1")
     (pin "2")
@@
     )
     (property "Datasheet" "~" (id 3) (at 134.62 147.32 0)
+      (effects (font (size 1.27 1.27)) hide)
+    )
+    (property "Do Not Place" "DNP" (id 4) (at 134.62 147.32 0)
+      (effects (font (size 1.27 1.27)) hide)
+    )
+    (property "LCSC" "DNP" (id 5) (at 134.62 147.32 0)
       (effects (font (size 1.27 1.27)) hide)
     )
@@
       (effects (font (size 1.27 1.27)) hide)
     )
+    (property "Alternate P/N" "MHPA3528RGBCT" (id 6) (at 43.18 71.12 0)
+      (effects (font (size 1.27 1.27)) hide)
+    )
+    (property "LCSC" "C409779" (id 7) (at 43.18 71.12 0)
+      (effects (font (size 1.27 1.27)) hide)
+    )
     (pin "1")
     (pin "2")
@@
       (effects (font (size 1.27 1.27)) hide)
     )
+    (property "Do Not Place" "DNP" (id 4) (at 158.75 184.15 0)
+      (effects (font (size 1.27 1.27)) hide)
+    )
+    (property "LCSC" "DNP" (id 5) (at 158.75 184.15 0)
+      (effects (font (size 1.27 1.27)) hide)
+    )

Commit message: Created Rev B1
Replaced buck regulator S-8581AA with AP63200 because of shortage
Parts:
- C15, C19, C23, C24, C29: LCSC P/N (none) -> C386079; LCSC Package (none) -> 0603; LCSC Specs (none) -> 1uF X7R 25V
- C16, C17, C18, C20, C21, C22, C25, C26, C28, C32: LCSC P/N (none) -> C77014; LCSC Package (none) -> 0402; LCSC Specs (none) -> 100nF X7R 16V
- C27, C30: LCSC P/N (none) -> C123543; LCSC Package (none) -> 0603; LCSC Specs (none) -> 20pF NP0/C0G 50V
- C31: LCSC P/N (none) -> C386019; LCSC Package (none) -> 0805; LCSC Specs (none) -> 10uF X7R 6.3V
- D7: Alternate P/N MHPA3528RGBCT -> (none); LCSC C409779 -> (none); LCSC P/N (none) -> C409779; LCSC Package (none) -> 3528; LCSC Specs (none) -> MHPA3528RGBCT
- D8, D9: LCSC C558429 -> (none); LCSC P/N (none) -> C558429; LCSC Package (none) -> SOT-23; LCSC Specs (none) -> TPCM1213A-01SO
- H1, H2, H3, H4, J3, R15, U4: LCSC DNP -> (none); LCSC P/N (none) -> DNP; LCSC Package (none) -> DNP; LCSC Specs (none) -> DNP
- J4: LCSC C124387 -> (none); LCSC P/N (none) -> C124387; LCSC Package (none) -> 2x5 P=2.54mm; LCSC Specs (none) -> B-2100S10P-B110
- L4, L5: LCSC C96995 -> (none); LCSC P/N (none) -> C96995; LCSC Package (none) -> 0603; LCSC Specs (none) -> UPZ1608E101-3R0TF
- R10: LCSC P/N (none) -> C114617; LCSC Package (none) -> 0603; LCSC Specs (none) -> 300R 1%
- R11: LCSC P/N (none) -> C22962; LCSC Package (none) -> 0603; LCSC Specs (none) -> 220R 1%
- R12: LCSC P/N (none) -> C22787; LCSC Package (none) -> 0603; LCSC Specs (none) -> 120R 1%
- R13, R14, R16: LCSC P/N (none) -> C98220; LCSC Package (none) -> 0603; LCSC Specs (none) -> 10K 1%
- U3: LCSC C3231235 -> (none); LCSC P/N (none) -> C3231235; LCSC Package (none) -> LQFP-64; LCSC Specs (none) -> M483SGCAE
- Y1: LCSC C91749 -> (none); LCSC P/N (none) -> C91749; LCSC Package (none) -> 3225; LCSC Specs (none) -> 12MHz 30ppm
