File: CAN-Acqusition-Module_Screen.kicad_sch (KiCad schematic)
At the start: 4 parts, among them U10 ERC13232FN-1

Commit message: Created Rev B1
Replaced buck regulator S-8581AA with AP63200 because of shortage
Parts:
- C59: LCSC P/N (none) -> C386079; LCSC Package (none) -> 0603; LCSC Specs (none) -> 1uF X7R 25V
- C60: LCSC P/N (none) -> C77014; LCSC Package (none) -> 0402; LCSC Specs (none) -> 100nF X7R 16V
- R72: LCSC P/N (none) -> C98220; LCSC Package (none) -> 0603; LCSC Specs (none) -> 10K 1%
- U10: LCSC P/N (none) -> DNP; LCSC Package (none) -> DNP; LCSC Specs (none) -> DNP
Changed lines of the file:
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@@
+      (effects (font (size 1.27 1.27)) hide)
+    )
+    (property "LCSC" "" (id 7) (at 104.14 74.93 0)
+      (effects (font (size 1.27 1.27)) hide)
+    )
+    (property "Specs" "" (id 8) (at 104.14 74.93 0)
+      (effects (font (size 1.27 1.27)) hide)
+    )
+    (property "LCSC P/N" "C386079" (id 9) (at 104.14 74.93 0)
+      (effects (font (size 1.27 1.27)) hide)
+    )
+    (property "LCSC Specs" "1uF X7R 25V" (id 10) (at 104.14 74.93 0)
+      (effects (font (size 1.27 1.27)) hide)
+    )
+    (property "LCSC Package" "0603" (id 11) (at 104.14 74.93 0)
       (effects (font (size 1.27 1.27)) hide)
     )
@@
       (effects (font (size 1.27 1.27)) hide)
     )
+    (property "LCSC" "" (id 7) (at 113.03 74.93 0)
+      (effects (font (size 1.27 1.27)) hide)
+    )
+    (property "Specs" "" (id 8) (at 113.03 74.93 0)
+      (effects (font (size 1.27 1.27)) hide)
+    )
+    (property "LCSC P/N" "C77014" (id 9) (at 113.03 74.93 0)
+      (effects (font (size 1.27 1.27)) hide)
+    )
+    (property "LCSC Specs" "100nF X7R 16V" (id 10) (at 113.03 74.93 0)
+      (effects (font (size 1.27 1.27)) hide)
+    )
+    (property "LCSC Package" "0402" (id 11) (at 113.03 74.93 0)
+      (effects (font (size 1.27 1.27)) hide)
+    )
     (pin "1")
     (pin "2")
@@
       (effects (font (size 1.27 1.27)) hide)
     )
+    (property "Specs" "" (id 7) (at 152.4 60.96 0)
+      (effects (font (size 1.27 1.27)) hide)
+    )
+    (property "LCSC" "" (id 8) (at 152.4 60.96 0)
+      (effects (font (size 1.27 1.27)) hide)
+    )
+    (property "LCSC P/N" "C98220" (id 9) (at 152.4 60.96 0)
+      (effects (font (size 1.27 1.27)) hide)
+    )
+    (property "LCSC Specs" "10K 1%" (id 10) (at 152.4 60.96 0)
+      (effects (font (size 1.27 1.27)) hide)
+    )
+    (property "LCSC Package" "0603" (id 11) (at 152.4 60.96 0)
+      (effects (font (size 1.27 1.27)) hide)
+    )
     (pin "1")
     (pin "2")
@@
       (effects (font (size 1.27 1.27)) hide)
     )
+    (property "LCSC P/N" "DNP" (id 6) (at 129.54 64.77 0)
+      (effects (font (size 1.27 1.27)) hide)
+    )
+    (property "LCSC Package" "DNP" (id 7) (at 129.54 64.77 0)
+      (effects (font (size 1.27 1.27)) hide)
+    )
+    (property "LCSC Specs" "DNP" (id 8) (at 129.54 64.77 0)
+      (effects (font (size 1.27 1.27)) hide)
+    )
